Commit message: refactor(fs3sw): unify launch flow and three-swerve integration
Add the new robot_forklift_simple_3sw Python package, update launch files to use the
shared xargs and bridge catalogs, and align the xacro model and example parameter files
with the current three-swerve solver conventions.

This includes the fs3sw wheel numbering, package imports, default config resolution and
the example Ground Vehicle Kinematics parameters now expected by the three-swerve node.

File: urdf/core.xacro (robot description, xacro)
@@ -1,10 +1,11 @@
 <?xml version="1.0"?>
 <!--
-The word 'fs3aw' is obtained from the combination of the words '(f)orklift', '(s)imple' and '(3) (a)ctive (w)heels'.
-This xacro file defines the 'core' version of the fs3aw robot, a base with 3 steerable wheels and a simple forklift.
+The word 'fs3sw' is obtained from the combination of the words '(f)orklift', '(s)imple' and '(3) (s)teerable
+(w)heels'.
+This xacro file defines the 'core' version of the fs3sw robot, a base with 3 steerable wheels and a simple forklift.
 No sensors or extra elements are included.
 -->
-<robot name="fs3aw_core" xmlns:xacro="http://www.ros.org/wiki/xacro" xmlns:gz="http://gazebosim.org/schema">
-  <xacro:property name="robot_forklift_simple_3aw_pkg_dir" value="$(find robot_forklift_simple_3aw)"/>
+<robot name="fs3sw_core" xmlns:xacro="http://www.ros.org/wiki/xacro" xmlns:gz="http://gazebosim.org/schema">
+  <xacro:property name="robot_forklift_simple_3sw_pkg_dir" value="$(find robot_forklift_simple_3sw)"/>
   <xacro:property name="robotics_description_pkg_dir"      value="$(find robotics_description)"/>
   <!-- ===================================================================== -->
@@ -24,5 +25,5 @@
   <xacro:arg name="use_sim_mode" default="False"/>
   <xacro:arg name="namespace"    default=""/>
-  <xacro:arg name="robot_name"   default="fs3aw"/>
+  <xacro:arg name="robot_name"   default="fs3sw"/>
   <!--
   File containing the simulation configuration for the platform.
@@ -31,5 +32,5 @@
   -->
   <xacro:arg name="sim_file"
-             default="${robot_forklift_simple_3aw_pkg_dir}/config/example_core_simulation.yaml"/>
+             default="${robot_forklift_simple_3sw_pkg_dir}/config/example_core_simulation.yaml"/>
   <!--
   Args for body
@@ -48,24 +49,24 @@
   <xacro:arg name="dist_to_wheels"         default="0.50"/>
   <xacro:arg name="alpha_deg"              default="154"/>
-  <xacro:arg name="body_mesh"              default="robot_forklift_simple_3aw/meshes/forklift_simple_3aw_base.stl"/>
+  <xacro:arg name="body_mesh"              default="robot_forklift_simple_3sw/meshes/forklift_simple_3aw_base.stl"/>
   <xacro:arg name="body_scale"             default="1.0 1.0 1.0"/>
   <xacro:arg name="body_color"             default="0.0 0.0 1.0 1.0"/>
   <!-- Wheels always use collision elements. Read the steerable_wheel macro for more details. -->
-  <xacro:arg name="st_wheel_use_inertial"  default="True"/>
-  <xacro:arg name="st_wheel_mass"          default="10.0"/>
-  <xacro:arg name="st_wheel_radius"        default="0.127"/>
-  <xacro:arg name="st_wheel_thickness"     default="0.082"/>
-  <xacro:arg name="st_wheel_color"         default="0.1 0.1 0.1 1.0"/>
+  <xacro:arg name="s_wheel_use_inertial"  default="True"/>
+  <xacro:arg name="s_wheel_mass"          default="10.0"/>
+  <xacro:arg name="s_wheel_radius"        default="0.127"/>
+  <xacro:arg name="s_wheel_thickness"     default="0.082"/>
+  <xacro:arg name="s_wheel_color"         default="0.1 0.1 0.1 1.0"/>
   <!--
   Note: If you want the wheel to be able to reach +-pi rad angle (+-180 degress), set limits to +-3.1416.
   pi = 3.141592654.... < 3.1416
   -->
-  <xacro:arg name="st_wheel_steerable_limits"      default="-3.1416 3.1416 100.0 100000.0"/>
-  <xacro:arg name="st_wheel_rotation_joint_limits" default="100.0 100000.0"/>
-  <xacro:arg name="st_wheel_max_contacts"          default="1"/>
-  <xacro:arg name="st_wheel_mu"                    default="0.05"/>
-  <xacro:arg name="st_wheel_mu2"                   default="0.5"/>
-  <xacro:arg name="st_wheel_slip1"                 default="0.005"/>
-  <xacro:arg name="st_wheel_slip2"                 default="0.0005"/>
+  <xacro:arg name="s_wheel_steerable_limits"      default="-3.1416 3.1416 100.0 100000.0"/>
+  <xacro:arg name="s_wheel_rotation_joint_limits" default="100.0 100000.0"/>
+  <xacro:arg name="s_wheel_max_contacts"          default="1"/>
+  <xacro:arg name="s_wheel_mu"                    default="0.05"/>
+  <xacro:arg name="s_wheel_mu2"                   default="0.5"/>
+  <xacro:arg name="s_wheel_slip1"                 default="0.005"/>
+  <xacro:arg name="s_wheel_slip2"                 default="0.0005"/>
   <!--
   Usually, forks are attached to the robot, on the front or the back side. The fork usually is a heavy body.
@@ -175,22 +176,22 @@
   <xacro:property name="body_color" value="$(arg body_color)"/>
   <!--
-  Wheel always use collision elements, which means 'st_wheel_use_collision' is always True.
-  Wheel always use a basic geometry for collision, which means 'st_wheel_use_c_mesh' is always False.
+  Wheel always use collision elements, which means 's_wheel_use_collision' is always True.
+  Wheel always use a basic geometry for collision, which means 's_wheel_use_c_mesh' is always False.
   Read the steerable_wheel macro for more details.
   -->
-  <xacro:property name="st_wheel_use_inertial" value="$(arg st_wheel_use_inertial)"/>
-  <xacro:property name="st_wheel_mass"                 value="$(arg st_wheel_mass)"/>
-  <xacro:property name="st_wheel_radius"               value="$(arg st_wheel_radius)"/>
-  <xacro:property name="st_wheel_thickness"            value="$(arg st_wheel_thickness)"/>
-  <xacro:property name="st_wheel_mesh"                 value=""/>
-  <xacro:property name="st_wheel_mesh_scale"           value="1.0 1.0 1.0"/>
-  <xacro:property name="st_wheel_mesh_origin"          value="0.0 0.0 0.0 0.0 0.0 0.0"/>
-  <xacro:property name="st_wheel_color"                value="$(arg st_wheel_color)"/>
-  <xacro:property name="st_wheel_steerable_joint_type" value="revolute"/>
+  <xacro:property name="s_wheel_use_inertial" value="$(arg s_wheel_use_inertial)"/>
+  <xacro:property name="s_wheel_mass"                 value="$(arg s_wheel_mass)"/>
+  <xacro:property name="s_wheel_radius"               value="$(arg s_wheel_radius)"/>
+  <xacro:property name="s_wheel_thickness"            value="$(arg s_wheel_thickness)"/>
+  <xacro:property name="s_wheel_mesh"                 value=""/>
+  <xacro:property name="s_wheel_mesh_scale"           value="1.0 1.0 1.0"/>
+  <xacro:property name="s_wheel_mesh_origin"          value="0.0 0.0 0.0 0.0 0.0 0.0"/>
+  <xacro:property name="s_wheel_color"                value="$(arg s_wheel_color)"/>
+  <xacro:property name="s_wheel_steerable_joint_type" value="revolute"/>
   <!--
   With this limits the steerable joint can rotate from [-pi, pi] radians.
   -->
-  <xacro:property name="st_wheel_steerable_joint_lower_limit"     value="${-pi}"/>
-  <xacro:property name="st_wheel_steerable_joint_upper_limit"     value="${pi}"/>
+  <xacro:property name="s_wheel_steerable_joint_lower_limit"     value="${-pi}"/>
+  <xacro:property name="s_wheel_steerable_joint_upper_limit"     value="${pi}"/>
   <!--
   Important:
@@ -206,12 +207,12 @@
   Read the macro 'steerable_wheel_macro.xacro' for more details about these limit parameters.
   -->
-  <xacro:property name="st_wheel_steerable_limits"                value="$(arg st_wheel_steerable_limits)"/>
-  <xacro:property name="st_wheel_rotation_joint_type"             value="continuous"/>
-  <xacro:property name="st_wheel_rotation_joint_limits"           value="$(arg st_wheel_rotation_joint_limits)"/>
-  <xacro:property name="st_wheel_max_contacts"                    value="$(arg st_wheel_max_contacts)"/>
-  <xacro:property name="st_wheel_mu"                              value="$(arg st_wheel_mu)"/>
-  <xacro:property name="st_wheel_mu2"                             value="$(arg st_wheel_mu2)"/>
-  <xacro:property name="st_wheel_slip1"                           value="$(arg st_wheel_slip1)"/>
-  <xacro:property name="st_wheel_slip2"                           value="$(arg st_wheel_slip2)"/>
+  <xacro:property name="s_wheel_steerable_limits"                value="$(arg s_wheel_steerable_limits)"/>
+  <xacro:property name="s_wheel_rotation_joint_type"             value="continuous"/>
+  <xacro:property name="s_wheel_rotation_joint_limits"           value="$(arg s_wheel_rotation_joint_limits)"/>
+  <xacro:property name="s_wheel_max_contacts"                    value="$(arg s_wheel_max_contacts)"/>
+  <xacro:property name="s_wheel_mu"                              value="$(arg s_wheel_mu)"/>
+  <xacro:property name="s_wheel_mu2"                             value="$(arg s_wheel_mu2)"/>
+  <xacro:property name="s_wheel_slip1"                           value="$(arg s_wheel_slip1)"/>
+  <xacro:property name="s_wheel_slip2"                           value="$(arg s_wheel_slip2)"/>
   <xacro:property name="fork_use_inertial"                        value="$(arg fork_use_inertial)"/>
   <!--
@@ -250,12 +251,12 @@
   <!-- Names for components -->
   <xacro:property name="base_name"                value="base"/>
+  <xacro:property name="steerable_wheel_0_name"   value="steerable_wheel_0"/>
   <xacro:property name="steerable_wheel_1_name"   value="steerable_wheel_1"/>
   <xacro:property name="steerable_wheel_2_name"   value="steerable_wheel_2"/>
-  <xacro:property name="steerable_wheel_3_name"   value="steerable_wheel_3"/>
   <xacro:property name="fork_name"                value="fork"/>
   <!-- Wheel numbering aligned with ground_vehicle_kinematics:
-       steerable_wheel_1 -> wheel on the robot X axis (x > 0 or x < 0 depending on geometry)
-       steerable_wheel_2 -> left wheel
-       steerable_wheel_3 -> right wheel
+       steerable_wheel_0 -> wheel on the robot X axis (x > 0 or x < 0 depending on geometry)
+       steerable_wheel_1 -> left wheel
+       steerable_wheel_2 -> right wheel
        Reference: package://ground_vehicle_kinematics/doc/kinematics_en.pdf -->
   <!-- ===================================================================== -->
@@ -333,5 +334,5 @@
   -->
   <!-- z-coordinate of each steerable wheel w.r.t it parent frame -->
-  <xacro:property name="z_st_wheel" value="${-body_ground_clearance + st_wheel_radius}"/>
+  <xacro:property name="z_s_wheel" value="${-body_ground_clearance + s_wheel_radius}"/>
   <xacro:property name="d" value="${float(dist_to_wheels)}"/>
   <xacro:property name="alpha" value="${radians(float(alpha_deg))}"/>
@@ -348,8 +349,8 @@
   - sin(-alpha) = -sin(alpha) -> y_right = -y_left
   -->
-  <xacro:property name="x_st_wheel_left"         value="${d * cos(alpha)}"/>
-  <xacro:property name="y_st_wheel_left"         value="${d * sin(alpha)}"/>
-  <xacro:property name="x_st_wheel_right"        value="${x_st_wheel_left}"/>
-  <xacro:property name="y_st_wheel_right"        value="${-y_st_wheel_left}"/>
+  <xacro:property name="x_s_wheel_left"         value="${d * cos(alpha)}"/>
+  <xacro:property name="y_s_wheel_left"         value="${d * sin(alpha)}"/>
+  <xacro:property name="x_s_wheel_right"        value="${x_s_wheel_left}"/>
+  <xacro:property name="y_s_wheel_right"        value="${-y_s_wheel_left}"/>
   <!--
   The longitudinal wheel is located on the x-axis, so its y coordinate is 0.
@@ -360,5 +361,5 @@
   equal to -d.
   -->
-  <xacro:property name="x_st_wheel_longitudinal" value="${d if float(alpha_deg) >= 90.0 else -d}"/>
+  <xacro:property name="x_s_wheel_longitudinal" value="${d if float(alpha_deg) >= 90.0 else -d}"/>
   <!--
   The steerable_wheel macro creates:
@@ -372,70 +373,70 @@
       parent=${prefix}${name}_steerable_link, child=${prefix}${name}_rotation_link
   -->
+  <xacro:steerable_wheel name="${steerable_wheel_0_name}"
+                         prefix="${robot_prefix}"
+                         parent_frame="${robot_prefix}${base_name}_link"
+                         use_visual="True"
+                         use_inertial="${s_wheel_use_inertial}"
+                         v_mesh="${s_wheel_mesh}"
+                         v_mesh_scale="${s_wheel_mesh_scale}"
+                         v_mesh_origin="${s_wheel_mesh_origin}"
+                         color="${s_wheel_color}"
+                         radius="${s_wheel_radius}"
+                         length="${s_wheel_thickness}"
+                         mass="${s_wheel_mass}"
+                         steerable_joint_type="${s_wheel_steerable_joint_type}"
+                         steerable_joint_steerable_limits="${s_wheel_steerable_limits}"
+                         rotation_joint_type="${s_wheel_rotation_joint_type}"
+                         rotation_joint_limits="${s_wheel_rotation_joint_limits}"
+                         max_contacts="${s_wheel_max_contacts}"
+                         mu="${s_wheel_mu}"
+                         mu2="${s_wheel_mu2}"
+                         slip1="${s_wheel_slip1}"
+                         slip2="${s_wheel_slip2}"
+                         joint_parent_fr_wheel_fr="${x_s_wheel_longitudinal} 0.0 ${z_s_wheel} 0.0 0.0 0.0"/>
   <xacro:steerable_wheel name="${steerable_wheel_1_name}"
                          prefix="${robot_prefix}"
                          parent_frame="${robot_prefix}${base_name}_link"
                          use_visual="True"
-                         use_inertial="${st_wheel_use_inertial}"
-                         v_mesh="${st_wheel_mesh}"
-                         v_mesh_scale="${st_wheel_mesh_scale}"
-                         v_mesh_origin="${st_wheel_mesh_origin}"
-                         color="${st_wheel_color}"
-                         radius="${st_wheel_radius}"
-                         length="${st_wheel_thickness}"
-                         mass="${st_wheel_mass}"
-                         steerable_joint_type="${st_wheel_steerable_joint_type}"
-                         steerable_joint_steerable_limits="${st_wheel_steerable_limits}"
-                         rotation_joint_type="${st_wheel_rotation_joint_type}"
-                         rotation_joint_limits="${st_wheel_rotation_joint_limits}"
-                         max_contacts="${st_wheel_max_contacts}"
-                         mu="${st_wheel_mu}"
-                         mu2="${st_wheel_mu2}"
-                         slip1="${st_wheel_slip1}"
-                         slip2="${st_wheel_slip2}"
-                         joint_parent_fr_wheel_fr="${x_st_wheel_longitudinal} 0.0 ${z_st_wheel} 0.0 0.0 0.0"/>
+                         use_inertial="${s_wheel_use_inertial}"
+                         v_mesh="${s_wheel_mesh}"
+                         v_mesh_scale="${s_wheel_mesh_scale}"
+                         v_mesh_origin="${s_wheel_mesh_origin}"
+                         color="${s_wheel_color}"
+                         radius="${s_wheel_radius}"
+                         length="${s_wheel_thickness}"
+                         mass="${s_wheel_mass}"
+                         steerable_joint_type="${s_wheel_steerable_joint_type}"
+                         steerable_joint_steerable_limits="${s_wheel_steerable_limits}"
+                         rotation_joint_type="${s_wheel_rotation_joint_type}"
+                         rotation_joint_limits="${s_wheel_rotation_joint_limits}"
+                         max_contacts="${s_wheel_max_contacts}"
+                         mu="${s_wheel_mu}"
+                         mu2="${s_wheel_mu2}"
+                         slip1="${s_wheel_slip1}"
+                         slip2="${s_wheel_slip2}"
+                         joint_parent_fr_wheel_fr="${x_s_wheel_left} ${y_s_wheel_left} ${z_s_wheel} 0.0 0.0 0.0"/>
   <xacro:steerable_wheel name="${steerable_wheel_2_name}"
                          prefix="${robot_prefix}"
                          parent_frame="${robot_prefix}${base_name}_link"
                          use_visual="True"
-                         use_inertial="${st_wheel_use_inertial}"
-                         v_mesh="${st_wheel_mesh}"
-                         v_mesh_scale="${st_wheel_mesh_scale}"
-                         v_mesh_origin="${st_wheel_mesh_origin}"
-                         color="${st_wheel_color}"
-                         radius="${st_wheel_radius}"
-                         length="${st_wheel_thickness}"
-                         mass="${st_wheel_mass}"
-                         steerable_joint_type="${st_wheel_steerable_joint_type}"
-                         steerable_joint_steerable_limits="${st_wheel_steerable_limits}"
-                         rotation_joint_type="${st_wheel_rotation_joint_type}"
-                         rotation_joint_limits="${st_wheel_rotation_joint_limits}"
-                         max_contacts="${st_wheel_max_contacts}"
-                         mu="${st_wheel_mu}"
-                         mu2="${st_wheel_mu2}"
-                         slip1="${st_wheel_slip1}"
-                         slip2="${st_wheel_slip2}"
-                         joint_parent_fr_wheel_fr="${x_st_wheel_left} ${y_st_wheel_left} ${z_st_wheel} 0.0 0.0 0.0"/>
-  <xacro:steerable_wheel name="${steerable_wheel_3_name}"
-                         prefix="${robot_prefix}"
-                         parent_frame="${robot_prefix}${base_name}_link"
-                         use_visual="True"
-                         use_inertial="${st_wheel_use_inertial}"
-                         v_mesh="${st_wheel_mesh}"
-                         v_mesh_scale="${st_wheel_mesh_scale}"
-                         v_mesh_origin="${st_wheel_mesh_origin}"
-                         color="${st_wheel_color}"
-                         radius="${st_wheel_radius}"
-                         length="${st_wheel_thickness}"
-                         mass="${st_wheel_mass}"
-                         steerable_joint_type="${st_wheel_steerable_joint_type}"
-                         steerable_joint_steerable_limits="${st_wheel_steerable_limits}"
-                         rotation_joint_type="${st_wheel_rotation_joint_type}"
-                         rotation_joint_limits="${st_wheel_rotation_joint_limits}"
-                         max_contacts="${st_wheel_max_contacts}"
-                         mu="${st_wheel_mu}"
-                         mu2="${st_wheel_mu2}"
-                         slip1="${st_wheel_slip1}"
-                         slip2="${st_wheel_slip2}"
-                         joint_parent_fr_wheel_fr="${x_st_wheel_right} ${y_st_wheel_right} ${z_st_wheel} 0.0 0.0 0.0"/>
+                         use_inertial="${s_wheel_use_inertial}"
+                         v_mesh="${s_wheel_mesh}"
+                         v_mesh_scale="${s_wheel_mesh_scale}"
+                         v_mesh_origin="${s_wheel_mesh_origin}"
+                         color="${s_wheel_color}"
+                         radius="${s_wheel_radius}"
+                         length="${s_wheel_thickness}"
+                         mass="${s_wheel_mass}"
+                         steerable_joint_type="${s_wheel_steerable_joint_type}"
+                         steerable_joint_steerable_limits="${s_wheel_steerable_limits}"
+                         rotation_joint_type="${s_wheel_rotation_joint_type}"
+                         rotation_joint_limits="${s_wheel_rotation_joint_limits}"
+                         max_contacts="${s_wheel_max_contacts}"
+                         mu="${s_wheel_mu}"
+                         mu2="${s_wheel_mu2}"
+                         slip1="${s_wheel_slip1}"
+                         slip2="${s_wheel_slip2}"
+                         joint_parent_fr_wheel_fr="${x_s_wheel_right} ${y_s_wheel_right} ${z_s_wheel} 0.0 0.0 0.0"/>
   <!-- ===================================================================== -->
   <!-- FORK -->
@@ -624,5 +625,5 @@
         <!-- Plugins to control the steerable joint of the steerable wheels. -->
         <plugin filename="gz-sim-joint-position-controller-system" name="gz::sim::systems::JointPositionController">
-          <joint_name>${robot_prefix}${steerable_wheel_1_name}_steerable_joint</joint_name>
+          <joint_name>${robot_prefix}${steerable_wheel_0_name}_steerable_joint</joint_name>
           <use_actuator_msg>true</use_actuator_msg>
           <!--
@@ -630,5 +631,5 @@
           Therefore, index 0 in the position array in the actuator message corresponds to the steerable wheel located
           on the x-axis of the robot frame, either with positive x-coordinate or negative x-coordinate.
-          Therefore, position at index 0 controls the orientation of steerable_wheel_1 in this robot.
+          Therefore, position at index 0 controls the orientation of steerable_wheel_0 in this robot.
           -->
           <actuator_number>0</actuator_number>
@@ -645,5 +646,5 @@
         </plugin>
         <plugin filename="gz-sim-joint-position-controller-system" name="gz::sim::systems::JointPositionController">
-          <joint_name>${robot_prefix}${steerable_wheel_2_name}_steerable_joint</joint_name>
+          <joint_name>${robot_prefix}${steerable_wheel_1_name}_steerable_joint</joint_name>
           <use_actuator_msg>true</use_actuator_msg>
           <!--
@@ -652,5 +653,5 @@
           opposite to steerable wheel 0, w.r.t the robot frame; i.e, if steerable wheel 0 is at positive x-coordinate,
           then steerable wheel 1 is at negative x-coordinate, and vice versa, and with positive y-coordinate.
-          Therefore, position at index 1 controls the orientation of steerable_wheel_2 in this robot.
+          Therefore, position at index 1 controls the orientation of steerable_wheel_1 in this robot.
           -->
           <actuator_number>1</actuator_number>
@@ -667,5 +668,5 @@
         </plugin>
         <plugin filename="gz-sim-joint-position-controller-system" name="gz::sim::systems::JointPositionController">
-          <joint_name>${robot_prefix}${steerable_wheel_3_name}_steerable_joint</joint_name>
+          <joint_name>${robot_prefix}${steerable_wheel_2_name}_steerable_joint</joint_name>
           <use_actuator_msg>true</use_actuator_msg>
           <!--
@@ -673,6 +674,6 @@
           Therefore, index 2 in the position array in the actuator message corresponds to the steerable wheel located
           opposite to steerable wheel 0, w.r.t the robot frame; i.e, if steerable wheel 0 is at positive x-coordinate,
-          then steerable wheel 1 is at negative x-coordinate, and vice versa, and with negative y-coordinate.
-          Therefore, position at index 2 controls the orientation of steerable_wheel_3 in this robot.
+          then steerable wheel 2 is at negative x-coordinate, and vice versa, and with negative y-coordinate.
+          Therefore, position at index 2 controls the orientation of steerable_wheel_2 in this robot.
           -->
           <actuator_number>2</actuator_number>
@@ -692,5 +693,5 @@
         <!-- Plugin to control the rotation joint of the steerable wheels. -->
         <plugin filename="gz-sim-joint-controller-system" name="gz::sim::systems::JointController">
-          <joint_name>${robot_prefix}${steerable_wheel_1_name}_rotation_joint</joint_name>
+          <joint_name>${robot_prefix}${steerable_wheel_0_name}_rotation_joint</joint_name>
           <!--
           use_force_commands: True to enable the controller implementation using force commands. If this parameter is
@@ -703,5 +704,5 @@
           Therefore, index 0 in the velocity array in the actuator message corresponds to the steerable wheel located
           on the x-axis of the robot frame, either with positive x-coordinate or negative x-coordinate.
-          Therefore, velocity at index 0 controls the velocity of steerable_wheel_1 in this robot.
+          Therefore, velocity at index 0 controls the velocity of steerable_wheel_0 in this robot.
           -->
           <actuator_number>0</actuator_number>
@@ -711,4 +712,19 @@
           <sub_topic> Sub topic to receive commands in. Defaults to "/model/<model_name>/<sub_topic>".
           -->
+          <initial_velocity>0.0</initial_velocity>
+        </plugin>
+        <plugin filename="gz-sim-joint-controller-system" name="gz::sim::systems::JointController">
+          <joint_name>${robot_prefix}${steerable_wheel_1_name}_rotation_joint</joint_name>
+          <use_force_commands>false</use_force_commands>
+          <use_actuator_msg>true</use_actuator_msg>
+          <!--
+          It is assumed that the ThreeSwerveKinematicsSolverRos is used to compute the wheel commands.
+          Therefore, index 1 in the velocity array in the actuator message corresponds to the steerable wheel located
+          opposite to steerable wheel 0, w.r.t the robot frame; i.e, if steerable wheel 0 is at positive x-coordinate,
+          then steerable wheel 1 is at negative x-coordinate, and vice versa, and with positive y-coordinate.
+          Therefore, velocity at index 1 controls the velocity of steerable_wheel_1 in this robot.
+          -->
+          <actuator_number>1</actuator_number>
+          <topic>${robot_namespace}/joint_commands/base</topic>
           <initial_velocity>0.0</initial_velocity>
         </plugin>
@@ -719,23 +735,8 @@
           <!--
           It is assumed that the ThreeSwerveKinematicsSolverRos is used to compute the wheel commands.
-          Therefore, index 1 in the velocity array in the actuator message corresponds to the steerable wheel located
-          opposite to steerable wheel 0, w.r.t the robot frame; i.e, if steerable wheel 0 is at positive x-coordinate,
-          then steerable wheel 1 is at negative x-coordinate, and vice versa, and with positive y-coordinate.
-          Therefore, velocity at index 1 controls the velocity of steerable_wheel_2 in this robot.
-          -->
-          <actuator_number>1</actuator_number>
-          <topic>${robot_namespace}/joint_commands/base</topic>
-          <initial_velocity>0.0</initial_velocity>
-        </plugin>
-        <plugin filename="gz-sim-joint-controller-system" name="gz::sim::systems::JointController">
-          <joint_name>${robot_prefix}${steerable_wheel_3_name}_rotation_joint</joint_name>
-          <use_force_commands>false</use_force_commands>
-          <use_actuator_msg>true</use_actuator_msg>
-          <!--
-          It is assumed that the ThreeSwerveKinematicsSolverRos is used to compute the wheel commands.
           Therefore, index 2 in the velocity array in the actuator message corresponds to the steerable wheel located
           opposite to steerable wheel 0, w.r.t the robot frame; i.e, if steerable wheel 0 is at positive x-coordinate,
           then steerable wheel 2 is at negative x-coordinate, and vice versa, and with negative y-coordinate.
-          Therefore, velocity at index 2 controls the velocity of steerable_wheel_3 in this robot.
+          Therefore, velocity at index 2 controls the velocity of steerable_wheel_2 in this robot.
           -->
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