Commit message: refactor(fs3sw): unify launch flow and three-swerve integration
Add the new robot_forklift_simple_3sw Python package, update launch files to use the
shared xargs and bridge catalogs, and align the xacro model and example parameter files
with the current three-swerve solver conventions.

This includes the fs3sw wheel numbering, package imports, default config resolution and
the example Ground Vehicle Kinematics parameters now expected by the three-swerve node.

File: urdf/v1.xacro (robot description, xacro)
@@ -1,19 +1,18 @@
 <?xml version="1.0"?>
 <!--
-The word 'fs3aw' is obtained from the combination of the words 'forklift' and 'artisteril', being 'artisteril' the
-company that manufactures the forklift robot.
-(f)ork(l)ift + (art)isteril -> fs3aw
-This xacro file defines the 'v1' version of the fs3aw robot, which a combination of the 'core' version plus:
+The word 'fs3sw' is obtained from the combination of the words '(f)orklift', '(s)imple' and '(3) (s)teerable
+(w)heels'.
+This xacro file defines the 'v1' version of the fs3sw robot, which is a combination of the 'core' version plus:
   - A top 3D LiDAR (RoboSense Helios 16P)
   - A top IMU (UM7)
   - A rear RGBD camera (Intel RealSense D435)
 -->
-<robot name="fs3aw_v1" xmlns:xacro="http://www.ros.org/wiki/xacro" xmlns:gz="http://gazebosim.org/schema">
-  <xacro:property name="robot_forklift_simple_3aw_pkg_dir"           value="$(find robot_forklift_simple_3aw)"/>
+<robot name="fs3sw_v1" xmlns:xacro="http://www.ros.org/wiki/xacro" xmlns:gz="http://gazebosim.org/schema">
+  <xacro:property name="robot_forklift_simple_3sw_pkg_dir"           value="$(find robot_forklift_simple_3sw)"/>
   <xacro:property name="robotics_description_pkg_dir"  value="$(find robotics_description)"/>
   <!-- ===================================================================== -->
   <!-- INCLUDES -->
   <!-- ===================================================================== -->
-  <xacro:include filename="${robot_forklift_simple_3aw_pkg_dir}/urdf/core.xacro"/>
+  <xacro:include filename="${robot_forklift_simple_3sw_pkg_dir}/urdf/core.xacro"/>
   <!--
   Properties imported from core.xacro and used in this file:

Commit message: refactor(urdf): load sim and bridge data from complete version configs
Update core.xacro and v1.xacro to consume the complete version-specific simulation and bridge YAML files.

Use rosgz_bridge_cfg to drive Gazebo plugin topics, align the v1 sensor plugins with the new bridge contract, and keep the rear camera block disabled while the camera redesign is still pending.

Reshape the example simulation YAML files to the same complete-per-version contract used by the launch flow.

File: urdf/core.xacro (robot description, xacro)
@@ -27,5 +27,5 @@
   <xacro:arg name="robot_name"   default="fs3sw"/>
   <!--
-  File containing the simulation configuration for the platform.
+  File containing the simulation configuration for the selected robot version.
   base = body + wheels.
   platform = base + fork.
@@ -33,4 +33,6 @@
   <xacro:arg name="sim_file"
              default="${robot_forklift_simple_3sw_pkg_dir}/config/example_core_simulation.yaml"/>
+  <xacro:arg name="rosgz_bridge_file"
+             default="${robot_forklift_simple_3sw_pkg_dir}/config/example_core_rosgz_bridge.yaml"/>
   <!--
   Args for body
@@ -105,23 +107,17 @@
   <xacro:make_prefix prop_id="robot_prefix" name="${robot_name}"/>
   <!--
-  If use_sim_mode is False (working in a real deployment), do not load the simulation configuration for the robot from
-  the simulation file.
+  If use_sim_mode is False (working in a real deployment), do not load the simulation configuration from the
+  simulation file.
   If use_sim_mode is True (working in simulation mode), and a configuration file is provided, load the simulation
   configuration from the file. If no configuration file is provided, use an empty configuration, so no gz-plugins are
   loaded.
   -->
-  <xacro:property name="sim_file" value="$(arg sim_file)"/>
-  <xacro:if value="${use_sim_mode}">
-    <xacro:if value="${sim_file != ''}">
-      <xacro:property name="sim_cfg" value="${xacro.load_yaml(sim_file)}"/>
-    </xacro:if>
-    <xacro:if value="${sim_file == ''}">
-      <xacro:property name="sim_cfg" value="${dict()}"/>
-    </xacro:if>
-  </xacro:if>
-  <xacro:unless value="${use_sim_mode}">
-    <xacro:property name="sim_cfg" value="${dict()}"/>
-  </xacro:unless>
-  <xacro:property name="body_use_inertial"     value="$(arg body_use_inertial)"/>
+  <xacro:property name="sim_file"          value="$(arg sim_file)"/>
+  <xacro:property name="rosgz_bridge_file" value="$(arg rosgz_bridge_file)"/>
+  <xacro:property name="sim_cfg"
+                  value="${xacro.load_yaml(sim_file) if use_sim_mode and sim_file != '' else dict()}"/>
+  <xacro:property name="rosgz_bridge_cfg"
+                  value="${xacro.load_yaml(rosgz_bridge_file) if use_sim_mode and rosgz_bridge_file != '' else dict()}"/>
+  <xacro:property name="body_use_inertial"  value="$(arg body_use_inertial)"/>
   <!--
   Base model overview:
@@ -490,18 +486,58 @@
   -->
   <xacro:if value="${use_sim_mode}">
-    <xacro:property name="base_sim_cfg" value="${sim_cfg.get('base', dict())}"/>
     <xacro:property name="base_velocity_controller_sim_cfg"
-                    value="${base_sim_cfg.get('velocity_controller', dict())}"/>
+                    value="${sim_cfg.get('base_velocity_controller', dict())}"/>
     <xacro:property name="base_pose_ground_truth_publisher_sim_cfg"
-                    value="${base_sim_cfg.get('pose_ground_truth_publisher', dict())}"/>
+                    value="${sim_cfg.get('base_pose_ground_truth_publisher', dict())}"/>
     <xacro:property name="steerable_wheel_steerable_joint_controller_sim_cfg"
-                    value="${base_sim_cfg.get('steerable_wheel_steerable_joint_controller', dict())}"/>
+                    value="${sim_cfg.get('base_steerable_wheel_steerable_joint_controller', dict())}"/>
     <xacro:property name="steerable_wheel_rotation_joint_controller_sim_cfg"
-                    value="${base_sim_cfg.get('steerable_wheel_rotation_joint_controller', dict())}"/>
-    <xacro:property name="fork_sim_cfg" value="${sim_cfg.get('fork', dict())}"/>
+                    value="${sim_cfg.get('base_steerable_wheel_rotation_joint_controller', dict())}"/>
     <xacro:property name="fork_position_controller_sim_cfg"
-                    value="${fork_sim_cfg.get('position_controller', dict())}"/>
+                    value="${sim_cfg.get('fork_position_controller', dict())}"/>
     <xacro:property name="joint_state_publisher_sim_cfg"
                     value="${sim_cfg.get('joint_state_publisher', dict())}"/>
+    <!-- 'bc_cfg' stands for (b)ridge (c)hannel (c)on(f)i(g)uration -->
+    <xacro:property name="bc_cfg_base_velocity_controller"
+                    value="${rosgz_bridge_cfg.get('base_velocity_controller', dict())}"/>
+    <xacro:property name="bc_cfg_base_pose_ground_truth_publisher"
+                    value="${rosgz_bridge_cfg.get('base_pose_ground_truth_publisher', dict())}"/>
+    <xacro:property name="bc_cfg_base_pose_ground_truth_publisher_tf"
+                    value="${rosgz_bridge_cfg.get('base_pose_ground_truth_publisher_tf', dict())}"/>
+    <xacro:property name="bc_cfg_base_steerable_wheel_command"
+                    value="${rosgz_bridge_cfg.get('base_steerable_wheel_command', dict())}"/>
+    <xacro:property name="bc_cfg_fork_position_controller"
+                    value="${rosgz_bridge_cfg.get('fork_position_controller', dict())}"/>
+    <xacro:property name="bc_cfg_joint_state_publisher"
+                    value="${rosgz_bridge_cfg.get('joint_state_publisher', dict())}"/>
+    <!--
+    # GZ topics for the plugins, with namespace handling.
+    If the topic name starts with '/', it is considered a global topic and used as is.
+    Otherwise, the topic name is prefixed with the robot namespace.
+    -->
+    <xacro:property name="base_velocity_controller_gz_topic"
+                    value="${bc_cfg_base_velocity_controller.get('gz_topic_name', 'cmd_vel')}"/>
+    <xacro:property name="base_velocity_controller_topic"
+                    value="${base_velocity_controller_gz_topic if base_velocity_controller_gz_topic.startswith('/') else robot_namespace + '/' + base_velocity_controller_gz_topic}"/>
+    <xacro:property name="base_pose_ground_truth_publisher_gz_topic"
+                    value="${bc_cfg_base_pose_ground_truth_publisher.get('gz_topic_name', 'base_pose_ground_truth')}"/>
+    <xacro:property name="base_pose_ground_truth_publisher_topic"
+                    value="${base_pose_ground_truth_publisher_gz_topic if base_pose_ground_truth_publisher_gz_topic.startswith('/') else robot_namespace + '/' + base_pose_ground_truth_publisher_gz_topic}"/>
+    <xacro:property name="base_pose_ground_truth_publisher_tf_gz_topic"
+                    value="${bc_cfg_base_pose_ground_truth_publisher_tf.get('gz_topic_name', 'tf_sim_world_fr_robot_root_fr')}"/>
+    <xacro:property name="base_pose_ground_truth_publisher_tf_topic"
+                    value="${base_pose_ground_truth_publisher_tf_gz_topic if base_pose_ground_truth_publisher_tf_gz_topic.startswith('/') else robot_namespace + '/' + base_pose_ground_truth_publisher_tf_gz_topic}"/>
+    <xacro:property name="base_steerable_wheel_command_gz_topic"
+                    value="${bc_cfg_base_steerable_wheel_command.get('gz_topic_name', 'joint_commands/base')}"/>
+    <xacro:property name="base_steerable_wheel_command_topic"
+                    value="${base_steerable_wheel_command_gz_topic if base_steerable_wheel_command_gz_topic.startswith('/') else robot_namespace + '/' + base_steerable_wheel_command_gz_topic}"/>
+    <xacro:property name="fork_position_controller_gz_topic"
+                    value="${bc_cfg_fork_position_controller.get('gz_topic_name', 'joint_commands/fork')}"/>
+    <xacro:property name="fork_position_controller_topic"
+                    value="${fork_position_controller_gz_topic if fork_position_controller_gz_topic.startswith('/') else robot_namespace + '/' + fork_position_controller_gz_topic}"/>
+    <xacro:property name="joint_state_publisher_gz_topic"
+                    value="${bc_cfg_joint_state_publisher.get('gz_topic_name', 'joint_states')}"/>
+    <xacro:property name="joint_state_publisher_topic"
+                    value="${joint_state_publisher_gz_topic if joint_state_publisher_gz_topic.startswith('/') else robot_namespace + '/' + joint_state_publisher_gz_topic}"/>
     <gazebo>
       <!--
@@ -523,5 +559,5 @@
         -->
         <plugin filename="gz-sim-velocity-control-system" name="gz::sim::systems::VelocityControl">
-          <topic>${robot_namespace}/cmd_vel</topic>
+          <topic>${base_velocity_controller_topic}</topic>
           <initial_linear>${initial_linear['x']} ${initial_linear['y']} ${initial_linear['z']}</initial_linear>
           <initial_angular>${initial_angular['x']} ${initial_angular['y']} ${initial_angular['z']}</initial_angular>
@@ -577,6 +613,4 @@
         <xacro:property name="pose_ground_truth_fixed_frame"
                         value="${base_pose_ground_truth_publisher_sim_cfg.get('fixed_frame', 'sim_world')}"/>
-        <xacro:property name="pose_ground_truth_tf_topic"
-                        value="${base_pose_ground_truth_publisher_sim_cfg.get('tf_topic', 'tf_sim_root_fr_robot_root_fr')}"/>
         <plugin filename="gz-sim-odometry-publisher-system" name="gz::sim::systems::OdometryPublisher">
           <odom_frame>${pose_ground_truth_fixed_frame}</odom_frame>
@@ -585,6 +619,6 @@
           <!--
           Custom topic on which this system will publish odometry messages.
-          The rosgz_bridge for this robot will not send this topic to ROS2, instead it will send the topic with
-          covariance.
+          The rosgz_bridge for this robot is configured not to send this topic to ROS2, instead it
+          will send the topic with covariance.
           -->
           <odom_topic>${robot_namespace}/base_pose_ground_truth_wo_cov</odom_topic>
@@ -599,9 +633,9 @@
           10.0 means a standard deviation of 10.0, and therefore a variance of 100.0.
           -->
-          <odom_covariance_topic>${robot_namespace}/base_pose_ground_truth</odom_covariance_topic>
+          <odom_covariance_topic>${base_pose_ground_truth_publisher_topic}</odom_covariance_topic>
           <!--
           Custom topic on which this system will publish the transform T:odometry_frame -> robot_base_frame.
           -->
-          <tf_topic>${robot_namespace}/${pose_ground_truth_tf_topic}</tf_topic>
+          <tf_topic>${base_pose_ground_truth_publisher_tf_topic}</tf_topic>
           <dimensions>2</dimensions> <!-- 2D (x, y, yaw) -->
           <!--
@@ -642,5 +676,5 @@
           -->
           <cmd_max>${steerable_wheel_steerable_joint_controller_sim_cfg.get('velocity', 100.0)}</cmd_max>
-          <topic>${robot_namespace}/joint_commands/base</topic>
+          <topic>${base_steerable_wheel_command_topic}</topic>
           <initial_position>0</initial_position>
         </plugin>
@@ -664,5 +698,5 @@
           -->
           <cmd_max>${steerable_wheel_steerable_joint_controller_sim_cfg.get('velocity', 100.0)}</cmd_max>
-          <topic>${robot_namespace}/joint_commands/base</topic>
+          <topic>${base_steerable_wheel_command_topic}</topic>
           <initial_position>0</initial_position>
         </plugin>
@@ -686,5 +720,5 @@
           -->
           <cmd_max>${steerable_wheel_steerable_joint_controller_sim_cfg.get('velocity', 100.0)}</cmd_max>
-          <topic>${robot_namespace}/joint_commands/base</topic>
+          <topic>${base_steerable_wheel_command_topic}</topic>
           <initial_position>0</initial_position>
         </plugin>
@@ -707,5 +741,5 @@
           -->
           <actuator_number>0</actuator_number>
-          <topic>${robot_namespace}/joint_commands/base</topic>
+          <topic>${base_steerable_wheel_command_topic}</topic>
           <!--
           NOT USED:
@@ -726,5 +760,5 @@
           -->
           <actuator_number>1</actuator_number>
-          <topic>${robot_namespace}/joint_commands/base</topic>
+          <topic>${base_steerable_wheel_command_topic}</topic>
           <initial_velocity>0.0</initial_velocity>
         </plugin>
@@ -741,5 +775,5 @@
           -->
           <actuator_number>2</actuator_number>
-          <topic>${robot_namespace}/joint_commands/base</topic>
+          <topic>${base_steerable_wheel_command_topic}</topic>
           <initial_velocity>0.0</initial_velocity>
         </plugin>
@@ -771,5 +805,5 @@
           <use_velocity_commands>true</use_velocity_commands>
           <cmd_max>${fork_position_controller_sim_cfg.get('velocity', 0.3)}</cmd_max>
-          <topic>${robot_namespace}/joint_commands/fork</topic>
+          <topic>${fork_position_controller_topic}</topic>
           <!-- Initial position of a joint. -->
           <initial_position>0</initial_position>
@@ -782,5 +816,5 @@
         -->
         <plugin filename="gz-sim-joint-state-publisher-system" name="gz::sim::systems::JointStatePublisher">
-          <topic>${robot_namespace}/joint_states</topic>
+          <topic>${joint_state_publisher_topic}</topic>
           <joint_name>${robot_prefix}${fork_name}_root_joint</joint_name>
           <joint_name>${robot_prefix}${steerable_wheel_0_name}_steerable_joint</joint_name>
