Commit message: feat(launch): rename bridge integration and wire v1 sensors
Replace the old rosgz bridge entrypoints and catalogs with the simplified bridge naming across launches, xargs, URDF arguments, and example configs.

Also wire the v1 rear camera through the RGBD-based setup, keep example simulation and bridge files aligned with the active sensor stack, and align example wheel radii with the robot defaults.

File: urdf/core.xacro (robot description, xacro)
@@ -33,6 +33,6 @@
   <xacro:arg name="sim_file"
              default="${robot_forklift_simple_3sw_pkg_dir}/config/example_core_simulation.yaml"/>
-  <xacro:arg name="rosgz_bridge_file"
-             default="${robot_forklift_simple_3sw_pkg_dir}/config/example_core_rosgz_bridge.yaml"/>
+  <xacro:arg name="bridge_file"
+             default="${robot_forklift_simple_3sw_pkg_dir}/config/example_core_bridge.yaml"/>
   <!--
   Args for body
@@ -113,10 +113,10 @@
   loaded.
   -->
-  <xacro:property name="sim_file"          value="$(arg sim_file)"/>
-  <xacro:property name="rosgz_bridge_file" value="$(arg rosgz_bridge_file)"/>
+  <xacro:property name="sim_file"    value="$(arg sim_file)"/>
+  <xacro:property name="bridge_file" value="$(arg bridge_file)"/>
   <xacro:property name="sim_cfg"
                   value="${xacro.load_yaml(sim_file) if use_sim_mode and sim_file != '' else dict()}"/>
-  <xacro:property name="rosgz_bridge_cfg"
-                  value="${xacro.load_yaml(rosgz_bridge_file) if use_sim_mode and rosgz_bridge_file != '' else dict()}"/>
+  <xacro:property name="bridge_cfg"
+                  value="${xacro.load_yaml(bridge_file) if use_sim_mode and bridge_file != '' else dict()}"/>
   <xacro:property name="body_use_inertial"  value="$(arg body_use_inertial)"/>
   <!--
@@ -498,17 +498,17 @@
     <xacro:property name="joint_state_publisher_sim_cfg"
                     value="${sim_cfg.get('joint_state_publisher', dict())}"/>
-    <!-- 'bc_cfg' stands for (b)ridge (c)hannel (c)on(f)i(g)uration -->
-    <xacro:property name="bc_cfg_base_velocity_controller"
-                    value="${rosgz_bridge_cfg.get('base_velocity_controller', dict())}"/>
-    <xacro:property name="bc_cfg_base_pose_ground_truth_publisher"
-                    value="${rosgz_bridge_cfg.get('base_pose_ground_truth_publisher', dict())}"/>
-    <xacro:property name="bc_cfg_base_pose_ground_truth_publisher_tf"
-                    value="${rosgz_bridge_cfg.get('base_pose_ground_truth_publisher_tf', dict())}"/>
-    <xacro:property name="bc_cfg_base_steerable_wheel_command"
-                    value="${rosgz_bridge_cfg.get('base_steerable_wheel_command', dict())}"/>
-    <xacro:property name="bc_cfg_fork_position_controller"
-                    value="${rosgz_bridge_cfg.get('fork_position_controller', dict())}"/>
-    <xacro:property name="bc_cfg_joint_state_publisher"
-                    value="${rosgz_bridge_cfg.get('joint_state_publisher', dict())}"/>
+    <!-- Bridge channel configurations -->
+    <xacro:property name="base_velocity_controller_bridge_channel_cfg"
+                    value="${bridge_cfg.get('base_velocity_controller', dict())}"/>
+    <xacro:property name="base_pose_ground_truth_publisher_bridge_channel_cfg"
+                    value="${bridge_cfg.get('base_pose_ground_truth_publisher', dict())}"/>
+    <xacro:property name="base_pose_ground_truth_publisher_tf_bridge_channel_cfg"
+                    value="${bridge_cfg.get('base_pose_ground_truth_publisher_tf', dict())}"/>
+    <xacro:property name="base_steerable_wheel_command_bridge_channel_cfg"
+                    value="${bridge_cfg.get('base_steerable_wheel_command', dict())}"/>
+    <xacro:property name="fork_position_controller_bridge_channel_cfg"
+                    value="${bridge_cfg.get('fork_position_controller', dict())}"/>
+    <xacro:property name="joint_state_publisher_bridge_channel_cfg"
+                    value="${bridge_cfg.get('joint_state_publisher', dict())}"/>
     <!--
     # GZ topics for the plugins, with namespace handling.
@@ -517,25 +517,25 @@
     -->
     <xacro:property name="base_velocity_controller_gz_topic"
-                    value="${bc_cfg_base_velocity_controller.get('gz_topic_name', 'cmd_vel')}"/>
+                    value="${base_velocity_controller_bridge_channel_cfg.get('gz_topic_name', 'cmd_vel')}"/>
     <xacro:property name="base_velocity_controller_topic"
                     value="${base_velocity_controller_gz_topic if base_velocity_controller_gz_topic.startswith('/') else robot_namespace + '/' + base_velocity_controller_gz_topic}"/>
     <xacro:property name="base_pose_ground_truth_publisher_gz_topic"
-                    value="${bc_cfg_base_pose_ground_truth_publisher.get('gz_topic_name', 'base_pose_ground_truth')}"/>
+                    value="${base_pose_ground_truth_publisher_bridge_channel_cfg.get('gz_topic_name', 'base_pose_ground_truth')}"/>
     <xacro:property name="base_pose_ground_truth_publisher_topic"
                     value="${base_pose_ground_truth_publisher_gz_topic if base_pose_ground_truth_publisher_gz_topic.startswith('/') else robot_namespace + '/' + base_pose_ground_truth_publisher_gz_topic}"/>
     <xacro:property name="base_pose_ground_truth_publisher_tf_gz_topic"
-                    value="${bc_cfg_base_pose_ground_truth_publisher_tf.get('gz_topic_name', 'tf_sim_world_fr_robot_root_fr')}"/>
+                    value="${base_pose_ground_truth_publisher_tf_bridge_channel_cfg.get('gz_topic_name', 'tf_sim_world_fr_robot_root_fr')}"/>
     <xacro:property name="base_pose_ground_truth_publisher_tf_topic"
                     value="${base_pose_ground_truth_publisher_tf_gz_topic if base_pose_ground_truth_publisher_tf_gz_topic.startswith('/') else robot_namespace + '/' + base_pose_ground_truth_publisher_tf_gz_topic}"/>
     <xacro:property name="base_steerable_wheel_command_gz_topic"
-                    value="${bc_cfg_base_steerable_wheel_command.get('gz_topic_name', 'joint_commands/base')}"/>
+                    value="${base_steerable_wheel_command_bridge_channel_cfg.get('gz_topic_name', 'joint_commands/base')}"/>
     <xacro:property name="base_steerable_wheel_command_topic"
                     value="${base_steerable_wheel_command_gz_topic if base_steerable_wheel_command_gz_topic.startswith('/') else robot_namespace + '/' + base_steerable_wheel_command_gz_topic}"/>
     <xacro:property name="fork_position_controller_gz_topic"
-                    value="${bc_cfg_fork_position_controller.get('gz_topic_name', 'joint_commands/fork')}"/>
+                    value="${fork_position_controller_bridge_channel_cfg.get('gz_topic_name', 'joint_commands/fork')}"/>
     <xacro:property name="fork_position_controller_topic"
                     value="${fork_position_controller_gz_topic if fork_position_controller_gz_topic.startswith('/') else robot_namespace + '/' + fork_position_controller_gz_topic}"/>
     <xacro:property name="joint_state_publisher_gz_topic"
-                    value="${bc_cfg_joint_state_publisher.get('gz_topic_name', 'joint_states')}"/>
+                    value="${joint_state_publisher_bridge_channel_cfg.get('gz_topic_name', 'joint_states')}"/>
     <xacro:property name="joint_state_publisher_topic"
                     value="${joint_state_publisher_gz_topic if joint_state_publisher_gz_topic.startswith('/') else robot_namespace + '/' + joint_state_publisher_gz_topic}"/>
@@ -619,5 +619,5 @@
           <!--
           Custom topic on which this system will publish odometry messages.
-          The rosgz_bridge for this robot is configured not to send this topic to ROS2, instead it
+          The bridge for this robot is configured not to send this topic to ROS2, instead it
           will send the topic with covariance.
           -->
@@ -625,5 +625,5 @@
           <!--
           Custom topic on which this system will publish odometry with covariance messages.
-          The rosgz_bridge for this robot will send this topic to ROS2.
+          The bridge for this robot will send this topic to ROS2.
           - The covariance is set as a diagonal matrix with the variance values set to the value of
           <gaussian_noise> squared.
