Commit message: refactor(robot_forklift_simple_3sw): reorganize launches and models around m1 and m2

File: urdf/includes/common.xacro (robot description, xacro)
@@ -1,10 +1,14 @@
 <?xml version="1.0"?>
 <!--
-The word 'fs3sw' is obtained from the combination of the words '(f)orklift', '(s)imple' and '(3) (s)teerable
-(w)heels'.
-This xacro file defines the 'core' model of the fs3sw robot, a base with 3 steerable wheels and a simple forklift.
-No sensors or extra elements are included.
+Common xacro file for the fs3sw robot family.
+THIS FILE IS NOT A COMPLETE ROBOT MODEL. IT IS MEANT TO BE INCLUDED FROM
+THE PUBLIC MODEL XACRO FILES, FOR EXAMPLE M1.XACRO AND M2.XACRO.
+The common robot contains:
+- the rectangular forklift base
+- the three steerable wheels
+- the simple fork
+- the Gazebo plugins that belong to that common mechanical structure
 -->
-<robot name="fs3sw_core" xmlns:xacro="http://www.ros.org/wiki/xacro" xmlns:gz="http://gazebosim.org/schema">
+<robot name="robot_forklift_simple_3sw_common" xmlns:xacro="http://www.ros.org/wiki/xacro" xmlns:gz="http://gazebosim.org/schema">
   <xacro:property name="robot_forklift_simple_3sw_pkg_dir" value="$(find robot_forklift_simple_3sw)"/>
   <xacro:property name="robotics_description_pkg_dir"      value="$(find robotics_description)"/>
@@ -35,5 +39,5 @@
   -->
   <xacro:arg name="sim_file"
-             default="${robot_forklift_simple_3sw_pkg_dir}/config/example_core_simulation.yaml"/>
+             default="${robot_forklift_simple_3sw_pkg_dir}/config/example_m1_simulation.yaml"/>
   <!--
   Args for body
@@ -52,5 +56,5 @@
   <xacro:arg name="dist_to_wheels"         default="0.50"/>
   <xacro:arg name="alpha_deg"              default="154"/>
-  <xacro:arg name="body_mesh"              default="robot_forklift_simple_3sw/meshes/forklift_simple_3aw_base.stl"/>
+  <xacro:arg name="body_mesh"              default="robot_forklift_simple_3sw/meshes/forklift_simple_3sw_base.stl"/>
   <xacro:arg name="body_scale"             default="1.0 1.0 1.0"/>
   <xacro:arg name="body_color"             default="0.0 0.0 1.0 1.0"/>
@@ -73,10 +77,9 @@
   <xacro:arg name="s_wheel_slip2"                 default="0.0005"/>
   <!--
-  Usually, forks are attached to the robot, on the front or the back side. The fork usually is a heavy body.
-  Attaching the fork with a considerable mass to the robot base, at the front or back, will affect the base's center
-  of mass, which will affect the robot's dynamics and stability in simulation, producing oscillations or even making the
-  robot to tip over.
-  Since simulation is used for kinematic behavior instead of dynamic behavior, the inertia of the fork, so even though
-  it is attached to the robot, the robot will move as it has no fork attached.
+  A fork can add a large mass far from the base center of mass.
+  If that inertia is included in simulation, the robot can oscillate or even tip over.
+  This robot is used mainly for kinematic simulation, not for accurate dynamic simulation.
+  For that reason, the fork inertia is disabled by default, so the fork is visible and attached
+  to the robot, but it does not change the simulated base dynamics.
   -->
   <xacro:arg name="fork_use_inertial"   default="False"/>
@@ -178,5 +181,4 @@
   <xacro:property name="s_wheel_mesh"                 value=""/>
   <xacro:property name="s_wheel_mesh_scale"           value="1.0 1.0 1.0"/>
-  <xacro:property name="s_wheel_mesh_origin"          value="0.0 0.0 0.0 0.0 0.0 0.0"/>
   <xacro:property name="s_wheel_color"                value="$(arg s_wheel_color)"/>
   <xacro:property name="s_wheel_steering_joint_type" value="revolute"/>
@@ -245,7 +247,8 @@
   operate in the range of [0.4, 0.6] m/s under load.
   -->
-  <xacro:property name="fork_limits" value="$(arg fork_limits)"/>
+  <xacro:property name="fork_limits"               value="$(arg fork_limits)"/>
   <!-- Distance from the ground to the bottom face of the tines. -->
-  <xacro:property name="fork_tines_rest_clearance"        value="$(arg fork_tines_rest_clearance)"/>
+  <xacro:property name="fork_tines_rest_clearance" value="$(arg fork_tines_rest_clearance)"/>
+  <xacro:property name="fork_open_tines"           value="True"/>
   <xacro:property name="robot_size_x" value="2.733"/>
   <xacro:property name="robot_size_y" value="0.774"/>
@@ -383,5 +386,4 @@
                          v_mesh="${s_wheel_mesh}"
                          v_mesh_scale="${s_wheel_mesh_scale}"
-                         v_mesh_origin="${s_wheel_mesh_origin}"
                          color="${s_wheel_color}"
                          radius="${s_wheel_radius}"
@@ -405,5 +407,4 @@
                          v_mesh="${s_wheel_mesh}"
                          v_mesh_scale="${s_wheel_mesh_scale}"
-                         v_mesh_origin="${s_wheel_mesh_origin}"
                          color="${s_wheel_color}"
                          radius="${s_wheel_radius}"
@@ -427,5 +428,4 @@
                          v_mesh="${s_wheel_mesh}"
                          v_mesh_scale="${s_wheel_mesh_scale}"
-                         v_mesh_origin="${s_wheel_mesh_origin}"
                          color="${s_wheel_color}"
                          radius="${s_wheel_radius}"
@@ -479,4 +479,5 @@
                      color="${fork_color}"
                      limits="${fork_limits}"
+                     open_tines="${fork_open_tines}"
                      joint_parent_fr_root_fr="${joint_base_fr_fork_fr_x} 0 ${joint_base_fr_fork_fr_z} 0 0 ${pi}"/>
   <!-- ===================================================================== -->
@@ -738,30 +739,4 @@
         </xacro:if>
       </xacro:if>
-      <!--
-      Define a 'JointStatePublisher' Gazebo plugin to report the states of the joints.
-      -->
-      <xacro:property name="joint_state_publisher_sim_cfg"
-                      value="${sim_cfg.get('joint_state_publisher', dict())}"/>
-      <xacro:if value="${joint_state_publisher_sim_cfg.get('enabled', False)}">
-        <xacro:property name="js_topic"
-                        value="${joint_state_publisher_sim_cfg.get('topic', '')}"/>
-        <!-- No topic, no Gazebo plugin -->
-        <xacro:if value="${js_topic != ''}">
-          <xacro:resolve_topic prop_id="resolved_js_topic"
-                               topic="${js_topic}"
-                               namespace="${robot_namespace}"/>
-          <xacro:plugin_joint_state_publisher topic="${resolved_js_topic}">
-            <joint_names>
-              <joint_name>${robot_prefix}${fork_name}_root_joint</joint_name>
-              <joint_name>${robot_prefix}${steerable_wheel_0_name}_steering_joint</joint_name>
-              <joint_name>${robot_prefix}${steerable_wheel_0_name}_rotation_joint</joint_name>
-              <joint_name>${robot_prefix}${steerable_wheel_1_name}_steering_joint</joint_name>
-              <joint_name>${robot_prefix}${steerable_wheel_1_name}_rotation_joint</joint_name>
-              <joint_name>${robot_prefix}${steerable_wheel_2_name}_steering_joint</joint_name>
-              <joint_name>${robot_prefix}${steerable_wheel_2_name}_rotation_joint</joint_name>
-            </joint_names>
-          </xacro:plugin_joint_state_publisher>
-        </xacro:if>
-      </xacro:if>
     </gazebo>
   </xacro:if>

Commit message: refactor(robot_forki3): align fork carriage and camera frames
Remove the local mast beam geometry from the common fork block and use the\nupdated fork_simple macro contract.\n\nMove the sensors1 fork cameras to the new carriage-link frame so their\nmount offsets follow the same pattern used by robot_vog.

File: urdf/includes/common.xacro (robot description, xacro)
@@ -408,7 +408,13 @@
   <xacro:property name="fork_upper_limit" value="${float(fork_limits_seq[1])}"/>
   <!--
-  Lower limit for the fork joint must be less than or equal to upper limit, and the limits must
-  satisfy lower <= 0 <= upper so that the joint can be at its rest position (q=0) without violating
-  the limits.
+  Lower limit for the fork joint must be less than or equal to upper limit.
+  Limits must satisfy lower <= 0 <= upper so that the joint can be initialized at its rest
+  position (q=0) without violating the range motion.
+    - If lower > 0, then q=0 is outside the motion limits and the fork will be initialized in an
+      invalid configuration.
+    - If upper < 0, then q=0 is outside the motion limits and the fork will be initialized in an
+      invalid configuration too.
+  The distance floor-to-bottom_face_carriage must (fork_rest_clearance) be > fork_lower_limit,
+  otherwise the fork would collide with the floor when moving to its lower limit position.
   -->
   <xacro:if value="${fork_lower_limit > fork_upper_limit}">
@@ -418,100 +424,15 @@
     ${xacro.fatal("xacro arg fork_limits must satisfy lower &lt;= 0 &lt;= upper, so q=0 is valid")}
   </xacro:if>
-  <xacro:if value="${fork_lower_limit &lt; -float(fork_rest_clearance)}">
+  <!--
+  Remember that after the fork limits checks above, the fork_lower_limit is negative, so the
+  condition is:
+  if abs(fork_lower_limit) > fork_rest_clearance -> the fork can collide with the floor when moving
+  to its lower limit position
+  -->
+  <xacro:if value="${python.abs(fork_lower_limit) > float(fork_rest_clearance)}">
     ${xacro.fatal("xacro args fork_limits and fork_rest_clearance are inconsistent: the allowed downward fork travel exceeds the rest clearance")}
   </xacro:if>
-  <!--
-  The mast is the vertical structure that supports the fork and guides its vertical motion.
-  `mast_left_beam` and `mast_right_beam` are the two vertical bars fixed to the robot body.
-  -->
-  <!-- mast_left_beam -->
-  <xacro:property name="mast_mass"     value="10.0"/>
-  <xacro:property name="mast_len_x"    value="0.03"/>
-  <xacro:property name="mast_len_y"    value="0.03"/>
-  <xacro:property name="mast_len_z"    value="${fork_upper_limit - fork_lower_limit}"/>
-  <xacro:property name="mast_origin_x" value="0"/>
-  <xacro:property name="mast_origin_y" value="0"/>
-  <xacro:property name="mast_origin_z" value="0"/>
-  <link name="${robot_prefix}${base_name}_mast_left_beam_link">
-    <xacro:if value="${fork_use_visual}">
-      <visual>
-        <geometry>
-          <box size="${mast_len_x} ${mast_len_y} ${mast_len_z}"/>
-        </geometry>
-        <origin rpy="0 0 0" xyz="${mast_origin_x} ${mast_origin_y} ${mast_origin_z}"/>
-        <material name="${robot_prefix}${fork_name}_color">
-          <color rgba="${fork_color}"/>
-        </material>
-      </visual>
-    </xacro:if>
-    <xacro:if value="${fork_use_collision}">
-      <collision>
-        <geometry>
-          <box size="${mast_len_x} ${mast_len_y} ${mast_len_z}"/>
-        </geometry>
-        <origin rpy="0 0 0" xyz="${mast_origin_x} ${mast_origin_y} ${mast_origin_z}"/>
-      </collision>
-    </xacro:if>
-    <xacro:if value="${fork_use_inertial}">
-      <xacro:solid_box_inertial mass="${mast_mass}"
-                                size="${mast_len_x} ${mast_len_y} ${mast_len_z}"
-                                origin="${mast_origin_x} ${mast_origin_y} ${mast_origin_z} 0 0 0"/>
-    </xacro:if>
-    <xacro:unless value="${fork_use_inertial}">
-      <xacro:null_inertia/>
-    </xacro:unless>
-  </link>
-  <xacro:property name="mast_mount_x" value="${-0.5 * (body_size_x + mast_len_x)}"/>
-  <xacro:property name="mast_mount_y" value="${0.5 * (body_size_y - mast_len_y)}"/>
-  <!--
-  mast goes from
-  inferior = -body_ground_clearance + fork_rest_clearance + fork_lower_limit
-  to
-  superior = inf + mast_len_z
-  The center is (sup + inf)/2 = (inf + mast_len_z + inf)/2 = inf + mast_len_z/2
-  -->
-  <xacro:property name="mast_mount_z" value="${-body_ground_clearance + fork_rest_clearance + fork_lower_limit + (0.5 * mast_len_z)}"/>
-  <joint name="${robot_prefix}${base_name}_mast_left_beam_joint" type="fixed">
-    <parent link="${robot_prefix}${base_name}_link"/>
-    <child link="${robot_prefix}${base_name}_mast_left_beam_link"/>
-    <origin rpy="0 0 0" xyz="${mast_mount_x} ${mast_mount_y} ${mast_mount_z}"/>
-  </joint>
-  <!-- mast_right_beam -->
-  <link name="${robot_prefix}${base_name}_mast_right_beam_link">
-    <xacro:if value="${fork_use_visual}">
-      <visual>
-        <geometry>
-          <box size="${mast_len_x} ${mast_len_y} ${mast_len_z}"/>
-        </geometry>
-        <origin rpy="0 0 0" xyz="${mast_origin_x} ${mast_origin_y} ${mast_origin_z}"/>
-        <material name="${robot_prefix}${fork_name}_color">
-          <color rgba="${fork_color}"/>
-        </material>
-      </visual>
-    </xacro:if>
-    <xacro:if value="${fork_use_collision}">
-      <collision>
-        <geometry>
-          <box size="${mast_len_x} ${mast_len_y} ${mast_len_z}"/>
-        </geometry>
-        <origin rpy="0 0 0" xyz="${mast_origin_x} ${mast_origin_y} ${mast_origin_z}"/>
-      </collision>
-    </xacro:if>
-    <xacro:if value="${fork_use_inertial}">
-      <xacro:solid_box_inertial mass="${mast_mass}"
-                                size="${mast_len_x} ${mast_len_y} ${mast_len_z}"
-                                origin="${mast_origin_x} ${mast_origin_y} ${mast_origin_z} 0 0 0"/>
-    </xacro:if>
-    <xacro:unless value="${fork_use_inertial}">
-      <xacro:null_inertia/>
-    </xacro:unless>
-  </link>
-  <joint name="${robot_prefix}${base_name}_mast_right_beam_joint" type="fixed">
-    <parent link="${robot_prefix}${base_name}_link"/>
-    <child link="${robot_prefix}${base_name}_mast_right_beam_link"/>
-    <origin rpy="0 0 0" xyz="${mast_mount_x} ${-mast_mount_y} ${mast_mount_z}"/>
-  </joint>
   <xacro:property name="fork_carriage_len_x"   value="0.03"/>
-  <xacro:property name="fork_carriage_mount_x" value="${mast_mount_x - (0.5*mast_len_x)}"/>
+  <xacro:property name="fork_carriage_mount_x" value="${-0.5 * body_size_x}"/>
   <xacro:property name="fork_carriage_mount_y" value="0"/>
   <xacro:property name="fork_carriage_mount_z" value="${-body_ground_clearance + fork_rest_clearance}"/>
@@ -529,6 +450,5 @@
                      color="${fork_color}"
                      use_c_mesh="${fork_use_c_mesh}"
-                     carriage_len_x="${fork_carriage_len_x}"
-                     carriage_len_y="${body_size_y}"
+                     carriage_size_x="${fork_carriage_len_x}"
                      limits="${fork_limits}"
                      joint_parent_fr_root_fr="${fork_carriage_mount_x} ${fork_carriage_mount_y} ${fork_carriage_mount_z} 0 0 ${pi}"/>

File: urdf/models/model_sensors1.xacro (robot description, xacro)
@@ -203,13 +203,11 @@
   (x = 0.002375 m, y = 0 m, z = 0.0125 m, R = 0 rad, P = 0 rad, Y = 0 rad).
   The bottom face of the mesh is touching the root frame of the camera.
-  Therefore, x_min = 0.002375 - (0.025053/2) m = -0.0101515 m.
-  Therefore, we have to move the root frame of the camera 0.0101515 m in the positive x-axis of
-  fork's root frame to have the back face of the camera aligned with the back face of the fork.
-  And, since the height of the union body that joins the tines of the fork is 6 cm, the root frame
-  of the camera has to be located at 6 cm in the z-axis of the fork's root frame.
-  -->
-  <xacro:property name="fork_rgbd_mount_x" value="0.0101515"/>
+  Therefore
+    x_min = 0.002375 - (0.025053/2) m = -0.0101515 m.
+    x_max = 0.002375 + (0.025053/2) m = 0.0148995 m.
+  -->
+  <xacro:property name="fork_rgbd_mount_x" value="${-0.0148995 - 0.01}"/>
   <xacro:property name="fork_rgbd_mount_y" value="0"/>
-  <xacro:property name="fork_rgbd_mount_z" value="${tine_size_z}"/>
+  <xacro:property name="fork_rgbd_mount_z" value="0"/>
   <xacro:realsense_d435_rgbd name="fork_camera"
                              prefix="${robot_prefix}"
@@ -291,7 +289,9 @@
                              sim_infra2_trigger_topic="${fork_camera_infra2_sim_trigger_topic}"/>
   <!--
-  The tine cameras are mounted near the front opening of each tine.
-  The x position uses the reference tine length and the fixed D435 body offset
-  used above. The y position places each camera at the center of its tine.
+  The tine cameras are mounted on `${robot_prefix}${fork_name}_carriage_link`.
+  The x position places each camera near the front opening of its tine.
+  The y position places each camera at the center of its tine.
+  The z position places each camera slightly above the bottom face of the tine, which usually
+  has 1 mm thickness.
   -->
   <!-- ===================================================================== -->
@@ -321,9 +321,8 @@
   tine_size_x - 0.0149 - 0.01 places the camera 1 cm behind the front opening of the left tine.
   -->
-  <xacro:property name="left_tine_rgbd_mount_x"
-                  value="${fork_carriage_len_x + tine_size_x - 0.0149 - 0.01}"/>
+  <xacro:property name="left_tine_rgbd_mount_x" value="${tine_size_x - 0.0149 - 0.01}"/>
   <xacro:property name="left_tine_rgbd_mount_y"
                   value="${0.5*(tine_separation + tine_size_y)}"/>
-  <xacro:property name="left_tine_rgbd_mount_z" value="0.001"/>
+  <xacro:property name="left_tine_rgbd_mount_z" value="${-tine_size_z + 0.001}"/>
   <xacro:realsense_d435_rgbd name="left_tine_camera"
                              prefix="${robot_prefix}"

Commit message: refactor(robot_forki3): [0408-01] align fork geometry with fork_simple
Update the common fork dimensions, pass carriage_size_z to the shared macro, move the tine cameras to the tine links, and point deps.repos to the matching robotics_description revision.

File: urdf/includes/common.xacro (robot description, xacro)
@@ -433,5 +433,6 @@
     ${xacro.fatal("xacro args fork_limits and fork_rest_clearance are inconsistent: the allowed downward fork travel exceeds the rest clearance")}
   </xacro:if>
-  <xacro:property name="fork_carriage_len_x"   value="0.03"/>
+  <xacro:property name="fork_carriage_len_x"   value="0.06"/>
+  <xacro:property name="fork_carriage_len_z"   value="0.06"/>
   <xacro:property name="fork_carriage_mount_x" value="${-0.5 * body_size_x}"/>
   <xacro:property name="fork_carriage_mount_y" value="0"/>
@@ -451,4 +452,5 @@
                      use_c_mesh="${fork_use_c_mesh}"
                      carriage_size_x="${fork_carriage_len_x}"
+                     carriage_size_z="${fork_carriage_len_z}"
                      limits="${fork_limits}"
                      joint_parent_fr_root_fr="${fork_carriage_mount_x} ${fork_carriage_mount_y} ${fork_carriage_mount_z} 0 0 ${pi}"/>

File: urdf/models/model_sensors1.xacro (robot description, xacro)
@@ -317,16 +317,15 @@
                                  sim_cfg="${left_tine_camera_infra2_sim_cfg}"/>
   <!--
-  The left tine camera is mounted in the carriage frame, not in `${robot_prefix}${base_name}_link`.
+  The left tine camera is mounted in the tine frame, not in `${robot_prefix}${base_name}_link`.
   The D435 front face is 0.0149 m in front of its root frame.
   tine_size_x - 0.0149 - 0.01 places the camera 1 cm behind the front opening of the left tine.
   -->
-  <xacro:property name="left_tine_rgbd_mount_x" value="${tine_size_x - 0.0149 - 0.01}"/>
-  <xacro:property name="left_tine_rgbd_mount_y"
-                  value="${0.5*(tine_separation + tine_size_y)}"/>
+  <xacro:property name="left_tine_rgbd_mount_x" value="${(0.5 * tine_size_x) - 0.0149 - 0.01}"/>
+  <xacro:property name="left_tine_rgbd_mount_y" value="0"/>
   <xacro:property name="left_tine_rgbd_mount_z" value="${-tine_size_z + 0.001}"/>
   <xacro:realsense_d435_rgbd name="left_tine_camera"
                              prefix="${robot_prefix}"
                              namespace="${robot_namespace}"
-                             parent_frame="${robot_prefix}${fork_name}_carriage_link"
+                             parent_frame="${robot_prefix}${fork_name}_left_tine_link"
                              use_visual="${left_tine_rgbd_use_visual}"
                              use_collision="${left_tine_rgbd_use_collision}"
@@ -426,5 +425,5 @@
   <!--
   The right tine camera uses the same x and z coordinates as the left tine camera.
-  The y coordinate is mirrored around the carriage center line.
+  The y coordinate is mirrored around the tine center line.
   -->
   <xacro:property name="right_tine_rgbd_mount_x" value="${left_tine_rgbd_mount_x}"/>
@@ -434,5 +433,5 @@
                              prefix="${robot_prefix}"
                              namespace="${robot_namespace}"
-                             parent_frame="${robot_prefix}${fork_name}_carriage_link"
+                             parent_frame="${robot_prefix}${fork_name}_right_tine_link"
                              use_visual="${right_tine_rgbd_use_visual}"
                              use_collision="${right_tine_rgbd_use_collision}"
