Commit message: refactor(sensors1): [0410-03] align with fork_simple updates
Update the sensors1 model to use the robotics_description revision that contains the latest fork_simple geometry and joint limit rules.

Keep the robot-specific fork validation focused on floor clearance and use -0.005 as the lower fork limit so q = 0 spawns 5 mm above the lower limit.

Also align the front top lidar mesh defaults with the repository policy and make model_sensors1.launch.py use the same generic model path construction as model_base.launch.py.

File: urdf/includes/common.xacro (robot description, xacro)
@@ -88,5 +88,5 @@
   <xacro:arg name="fork_color"          default="0.1 0.1 0.1 1.0"/>
   <xacro:arg name="fork_use_c_mesh"     default="True"/>
-  <xacro:arg name="fork_limits"         default="-0.01 0.8 0.5 20000.0"/>
+  <xacro:arg name="fork_limits"         default="-0.005 0.8 0.5 20000.0"/>
   <xacro:arg name="fork_rest_clearance" default="0.03"/>
   <!-- Create properties from args for easy manipulation. -->
@@ -402,28 +402,19 @@
     ${xacro.fatal("xacro arg fork_limits must contain exactly 4 values: lower upper velocity effort")}
   </xacro:if>
-  <xacro:property name="fork_lower_limit" value="${float(fork_limits_seq[0])}"/>
-  <xacro:property name="fork_upper_limit" value="${float(fork_limits_seq[1])}"/>
-  <!--
-  Lower limit for the fork joint must be less than or equal to upper limit.
-  Limits must satisfy lower <= 0 <= upper so that the joint can be initialized at its rest
-  position (q=0) without violating the range motion.
-    - If lower > 0, then q=0 is outside the motion limits and the fork will be initialized in an
-      invalid configuration.
-    - If upper < 0, then q=0 is outside the motion limits and the fork will be initialized in an
-      invalid configuration too.
+  <!--
+  The fork_simple macro checks that the fork limits are valid for the fork joint.
+  This module only checks the part that is specific to the robot installation.
+  fork_lower_limit must be less than or equal to zero so that this installation allows downward
+  fork motion from the spawned joint position.
   The distance floor-to-bottom_face_carriage must (fork_rest_clearance) be > fork_lower_limit,
   otherwise the fork would collide with the floor when moving to its lower limit position.
   -->
-  <xacro:if value="${fork_lower_limit > fork_upper_limit}">
-    ${xacro.fatal("xacro arg fork_limits must satisfy lower &lt;= upper")}
+  <xacro:property name="fork_lower_limit" value="${float(fork_limits_seq[0])}"/>
+  <xacro:if value="${fork_lower_limit > 0.0}">
+    ${xacro.fatal("xacro arg fork_limits must satisfy lower &lt;= 0 for this robot installation")}
   </xacro:if>
-  <xacro:if value="${fork_lower_limit > 0.0 or fork_upper_limit &lt; 0.0}">
-    ${xacro.fatal("xacro arg fork_limits must satisfy lower &lt;= 0 &lt;= upper, so q=0 is valid")}
-  </xacro:if>
-  <!--
-  Remember that after the fork limits checks above, the fork_lower_limit is negative, so the
-  condition is:
-  if abs(fork_lower_limit) > fork_rest_clearance -> the fork can collide with the floor when moving
-  to its lower limit position
+  <!--
+  At this point fork_lower_limit is less than or equal to zero, so the downward fork travel is
+  abs(fork_lower_limit).
   -->
   <xacro:if value="${python.abs(fork_lower_limit) > float(fork_rest_clearance)}">

File: urdf/models/model_sensors1.xacro (robot description, xacro)
@@ -104,5 +104,5 @@
   <xacro:arg name="front_top_lidar_use_collision"      default="True"/>
   <xacro:arg name="front_top_lidar_use_inertial"       default="True"/>
-  <xacro:arg name="front_top_lidar_use_v_mesh"         default="False"/>
+  <xacro:arg name="front_top_lidar_use_v_mesh"         default="True"/>
   <!--
   The low resolution mesh has its own color.
@@ -113,5 +113,5 @@
   <!-- Use shape instead of mesh for collision by default. -->
   <xacro:arg name="front_top_lidar_use_c_mesh"         default="False"/>
-  <xacro:arg name="front_top_lidar_c_mesh_use_low_res" default="False"/>
+  <xacro:arg name="front_top_lidar_c_mesh_use_low_res" default="True"/>
   <!--
   tilt_angle = pitch = 20 deg = 0.34906585 rad
