Commit message: chore: align robot_forki3 package rules
Migrate the package to ament_cmake_python, update launch/config organization, add package tests and align lint configuration with the agreed ROS 2 package rules.

File: urdf/models/model_sensors1.xacro (robot description, xacro)
@@ -144,5 +144,5 @@
       c_mesh_use_low_res="${front_top_lidar_c_mesh_use_low_res}"
       joint_parent_fr_root_fr="${front_top_lidar_mount}"
-      sim_lidar_enabled="${use_sim_mode and front_top_lidar_sim_enabled}"
+      sim_lidar_enabled="${sim_file != '' and front_top_lidar_sim_enabled}"
       sim_lidar_always_on="${front_top_lidar_sim_always_on}"
       sim_lidar_visualize="${front_top_lidar_sim_visualize}"
@@ -154,5 +154,5 @@
       sim_lidar_dist_span="${front_top_lidar_sim_dist_span}"
       sim_lidar_gaussian_noise="${front_top_lidar_sim_gaussian_noise}"
-      sim_imu_enabled="${use_sim_mode and front_top_lidar_imu_sim_enabled}"
+      sim_imu_enabled="${sim_file != '' and front_top_lidar_imu_sim_enabled}"
       sim_imu_use_gravity="${front_top_lidar_imu_sim_use_gravity}"
       sim_imu_always_on="${front_top_lidar_imu_sim_always_on}"
@@ -232,5 +232,5 @@
       c_mesh_use_low_res="${back_top_lidar_c_mesh_use_low_res}"
       joint_parent_fr_root_fr="${back_top_lidar_mount}"
-      sim_lidar_enabled="${use_sim_mode and back_top_lidar_sim_enabled}"
+      sim_lidar_enabled="${sim_file != '' and back_top_lidar_sim_enabled}"
       sim_lidar_always_on="${back_top_lidar_sim_always_on}"
       sim_lidar_visualize="${back_top_lidar_sim_visualize}"
@@ -242,5 +242,5 @@
       sim_lidar_dist_span="${back_top_lidar_sim_dist_span}"
       sim_lidar_gaussian_noise="${back_top_lidar_sim_gaussian_noise}"
-      sim_imu_enabled="${use_sim_mode and back_top_lidar_imu_sim_enabled}"
+      sim_imu_enabled="${sim_file != '' and back_top_lidar_imu_sim_enabled}"
       sim_imu_use_gravity="${back_top_lidar_imu_sim_use_gravity}"
       sim_imu_always_on="${back_top_lidar_imu_sim_always_on}"
@@ -275,5 +275,5 @@
     = -0.06 + 0.152 + 0.20 = 0.292
   -->
-  <xacro:arg name="back_bottom_lidar_mount"              default= "-0.7025 0 0.292 3.141592654 0 3.141592654"/>
+  <xacro:arg name="back_bottom_lidar_mount"              default="-0.7025 0 0.292 3.141592654 0 3.141592654"/>
   <xacro:property name="back_bottom_lidar_use_visual"         value="$(arg back_bottom_lidar_use_visual)"/>
   <xacro:property name="back_bottom_lidar_use_collision"      value="$(arg back_bottom_lidar_use_collision)"/>
@@ -311,14 +311,14 @@
     c_mesh_use_low_res="${back_bottom_lidar_c_mesh_use_low_res}"
     joint_parent_fr_root_fr="${back_bottom_lidar_mount}"
-    sim_lidar_enabled="${use_sim_mode and back_bottom_lidar_sim_enabled}"
-    sim_lidar_always_on="${back_bottom_lidar_sim_always_on}"
-    sim_lidar_visualize="${back_bottom_lidar_sim_visualize}"
-    sim_lidar_update_rate="${back_bottom_lidar_sim_update_rate}"
-    sim_lidar_hor_fov_deg="${back_bottom_lidar_sim_hor_fov_deg}"
-    sim_lidar_hor_res_deg="${back_bottom_lidar_sim_hor_res_deg}"
-    sim_lidar_dist_span="${back_bottom_lidar_sim_dist_span}"
-    sim_lidar_gaussian_noise="${back_bottom_lidar_sim_gaussian_noise}"
+    sim_enabled="${sim_file != '' and back_bottom_lidar_sim_enabled}"
+    sim_always_on="${back_bottom_lidar_sim_always_on}"
+    sim_visualize="${back_bottom_lidar_sim_visualize}"
+    sim_update_rate="${back_bottom_lidar_sim_update_rate}"
+    sim_hor_fov_deg="${back_bottom_lidar_sim_hor_fov_deg}"
+    sim_hor_res_deg="${back_bottom_lidar_sim_hor_res_deg}"
+    sim_dist_span="${back_bottom_lidar_sim_dist_span}"
+    sim_gaussian_noise="${back_bottom_lidar_sim_gaussian_noise}"
     namespace="${robot_namespace}"
-    sim_lidar_topic="${back_bottom_lidar_sim_topic}"/>
+    sim_topic="${back_bottom_lidar_sim_topic}"/>
   <!-- ===================================================================== -->
   <!-- FORK CAMERA: REALSENSE D435 -->
@@ -373,6 +373,6 @@
                              use_c_mesh="${fork_rgbd_use_c_mesh}"
                              joint_parent_fr_root_fr="${fork_rgbd_mount_x} ${fork_rgbd_mount_y} ${fork_rgbd_mount_z} 0 0 0"
-                             use_sensor_frames_and_joints="${use_sim_mode}"
-                             sim_rgbd_enabled="${use_sim_mode and fork_camera_rgbd_sim_enabled}"
+                             use_sensor_frames_and_joints="${sim_file != ''}"
+                             sim_rgbd_enabled="${sim_file != '' and fork_camera_rgbd_sim_enabled}"
                              sim_rgbd_use_gravity="${fork_camera_rgbd_sim_use_gravity}"
                              sim_rgbd_always_on="${fork_camera_rgbd_sim_always_on}"
@@ -394,5 +394,5 @@
                              sim_rgbd_distortion_center="${fork_camera_rgbd_sim_distortion_center}"
                              sim_rgbd_gaussian_noise="${fork_camera_rgbd_sim_gaussian_noise}"
-                             sim_infra1_enabled="${use_sim_mode and fork_camera_infra1_sim_enabled}"
+                             sim_infra1_enabled="${sim_file != '' and fork_camera_infra1_sim_enabled}"
                              sim_infra1_use_gravity="${fork_camera_infra1_sim_use_gravity}"
                              sim_infra1_always_on="${fork_camera_infra1_sim_always_on}"
@@ -413,5 +413,5 @@
                              sim_infra1_distortion_center="${fork_camera_infra1_sim_distortion_center}"
                              sim_infra1_gaussian_noise="${fork_camera_infra1_sim_gaussian_noise}"
-                             sim_infra2_enabled="${use_sim_mode and fork_camera_infra2_sim_enabled}"
+                             sim_infra2_enabled="${sim_file != '' and fork_camera_infra2_sim_enabled}"
                              sim_infra2_use_gravity="${fork_camera_infra2_sim_use_gravity}"
                              sim_infra2_always_on="${fork_camera_infra2_sim_always_on}"
@@ -440,5 +440,5 @@
                              sim_infra2_camera_info_topic="${fork_camera_infra2_sim_info_topic}"
                              sim_infra2_trigger_topic="${fork_camera_infra2_sim_trigger_topic}"/>
-  <xacro:if value="${use_sim_mode}">
+  <xacro:if value="${sim_file != ''}">
     <gazebo>
       <!--
@@ -450,5 +450,8 @@
         <xacro:property name="js_topic"
                         value="${joint_state_publisher_sim_cfg.get('topic', '')}"/>
-        <!-- No topic, no Gazebo plugin -->
+        <xacro:if value="${js_topic == ''}">
+          ${xacro.fatal(
+            "joint_state_publisher.topic is required when joint_state_publisher.enabled is true.")}
+        </xacro:if>
         <xacro:if value="${js_topic != ''}">
           <xacro:resolve_topic prop_id="resolved_js_topic"
