Commit message: refactor(sensors1): [0416-03] remove left and right tine cameras
Remove Intel RealSense D435 cameras from left and right fork tines.

Changes:
- Remove left_tine_camera and right_tine_camera definitions from URDF
- Remove tine camera xacro arguments from model_sensors1.yaml
- Remove tine camera bridge configurations
- Remove tine camera simulation configurations

This eliminates 762 lines across 4 files including URDF macros,
xacro arguments, bridge mappings, and simulation plugin settings.

File: urdf/models/model_sensors1.xacro (robot description, xacro)
@@ -5,6 +5,4 @@
   - A top 3D LiDAR with integrated IMU (RoboSense Airy)
   - A rear RGBD camera (Intel RealSense D435)
-  - A left tine RGBD camera (Intel RealSense D435)
-  - A right tine RGBD camera (Intel RealSense D435)
 -->
 <robot name="forki3_sensors1" xmlns:xacro="http://www.ros.org/wiki/xacro" xmlns:gz="http://gazebosim.org/schema">
@@ -31,18 +29,4 @@
   <!-- Use shape instead of mesh for collision by default. -->
   <xacro:arg name="fork_rgbd_use_c_mesh"       default="False"/>
-  <xacro:arg name="left_tine_rgbd_use_visual"    default="True"/>
-  <xacro:arg name="left_tine_rgbd_use_collision" default="True"/>
-  <xacro:arg name="left_tine_rgbd_use_inertial"  default="True"/>
-  <xacro:arg name="left_tine_rgbd_use_v_mesh"    default="True"/>
-  <xacro:arg name="left_tine_rgbd_color"         default="0.5 0.5 0.5 1.0"/>
-  <!-- Use shape instead of mesh for collision by default. -->
-  <xacro:arg name="left_tine_rgbd_use_c_mesh"    default="False"/>
-  <xacro:arg name="right_tine_rgbd_use_visual"    default="True"/>
-  <xacro:arg name="right_tine_rgbd_use_collision" default="True"/>
-  <xacro:arg name="right_tine_rgbd_use_inertial"  default="True"/>
-  <xacro:arg name="right_tine_rgbd_use_v_mesh"    default="True"/>
-  <xacro:arg name="right_tine_rgbd_color"         default="0.5 0.5 0.5 1.0"/>
-  <!-- Use shape instead of mesh for collision by default. -->
-  <xacro:arg name="right_tine_rgbd_use_c_mesh"    default="False"/>
   <!-- ===================================================================== -->
   <!-- DEFINITION OF PROPERTIES -->
@@ -456,224 +440,4 @@
                              sim_infra2_camera_info_topic="${fork_camera_infra2_sim_info_topic}"
                              sim_infra2_trigger_topic="${fork_camera_infra2_sim_trigger_topic}"/>
-  <!--
-  The tine cameras are mounted on `${robot_prefix}${fork_name}_carriage_link`.
-  The x position places each camera near the front opening of its tine.
-  The y position places each camera at the center of its tine.
-  The z position places each camera slightly above the bottom face of the tine, which usually
-  has 1 mm thickness.
-  -->
-  <!-- ===================================================================== -->
-  <!-- LEFT TINE CAMERA: REALSENSE D435 -->
-  <!-- ===================================================================== -->
-  <xacro:property name="left_tine_rgbd_use_visual"       value="$(arg left_tine_rgbd_use_visual)"/>
-  <xacro:property name="left_tine_rgbd_use_collision"    value="$(arg left_tine_rgbd_use_collision)"/>
-  <xacro:property name="left_tine_rgbd_use_inertial"     value="$(arg left_tine_rgbd_use_inertial)"/>
-  <xacro:property name="left_tine_rgbd_use_v_mesh"       value="$(arg left_tine_rgbd_use_v_mesh)"/>
-  <xacro:property name="left_tine_rgbd_color"            value="$(arg left_tine_rgbd_color)"/>
-  <xacro:property name="left_tine_rgbd_use_c_mesh"       value="$(arg left_tine_rgbd_use_c_mesh)"/>
-  <xacro:property name="left_tine_camera_rgbd_sim_cfg"   value="${sim_cfg.get('left_tine_camera_rgbd', dict())}"/>
-  <xacro:property name="left_tine_camera_infra1_sim_cfg" value="${sim_cfg.get('left_tine_camera_infra1', dict())}"/>
-  <xacro:property name="left_tine_camera_infra2_sim_cfg" value="${sim_cfg.get('left_tine_camera_infra2', dict())}"/>
-  <!-- Set properties for the `rgbd_camera` Gazebo plugin associated to the left tine camera. -->
-  <xacro:set_props_plugin_camera_rgbd prop_prefix="left_tine_camera_rgbd_sim"
-                                      sim_cfg="${left_tine_camera_rgbd_sim_cfg}"/>
-  <!-- Set properties for the first infrared Gazebo plugin in the left tine camera. -->
-  <xacro:set_props_plugin_camera prop_prefix="left_tine_camera_infra1_sim"
-                                 sim_cfg="${left_tine_camera_infra1_sim_cfg}"/>
-  <!-- Set properties for the second infrared Gazebo plugin in the left tine camera. -->
-  <xacro:set_props_plugin_camera prop_prefix="left_tine_camera_infra2_sim"
-                                 sim_cfg="${left_tine_camera_infra2_sim_cfg}"/>
-  <!--
-  The left tine camera is mounted in the tine frame, not in `${robot_prefix}${base_name}_link`.
-  The D435 front face is 0.0149 m in front of its root frame.
-  tine_size_x - 0.0149 - 0.01 places the camera 1 cm behind the front opening of the left tine.
-  -->
-  <xacro:property name="left_tine_rgbd_mount_x" value="${(0.5 * tine_size_x) - 0.0149 - 0.01}"/>
-  <xacro:property name="left_tine_rgbd_mount_y" value="0"/>
-  <xacro:property name="left_tine_rgbd_mount_z" value="${-tine_size_z + 0.001}"/>
-  <xacro:realsense_d435_rgbd name="left_tine_camera"
-                             prefix="${robot_prefix}"
-                             namespace="${robot_namespace}"
-                             parent_frame="${robot_prefix}${fork_name}_left_tine_link"
-                             use_visual="${left_tine_rgbd_use_visual}"
-                             use_collision="${left_tine_rgbd_use_collision}"
-                             use_inertial="${left_tine_rgbd_use_inertial}"
-                             use_v_mesh="${left_tine_rgbd_use_v_mesh}"
-                             color="${left_tine_rgbd_color}"
-                             use_c_mesh="${left_tine_rgbd_use_c_mesh}"
-                             joint_parent_fr_root_fr="${left_tine_rgbd_mount_x} ${left_tine_rgbd_mount_y} ${left_tine_rgbd_mount_z} 0.0 0.0 0.0"
-                             use_sensor_frames_and_joints="${use_sim_mode}"
-                             sim_rgbd_enabled="${use_sim_mode and left_tine_camera_rgbd_sim_enabled}"
-                             sim_rgbd_use_gravity="${left_tine_camera_rgbd_sim_use_gravity}"
-                             sim_rgbd_always_on="${left_tine_camera_rgbd_sim_always_on}"
-                             sim_rgbd_visualize="${left_tine_camera_rgbd_sim_visualize}"
-                             sim_rgbd_enable_metrics="${left_tine_camera_rgbd_sim_enable_metrics}"
-                             sim_rgbd_save="${left_tine_camera_rgbd_sim_save}"
-                             sim_rgbd_triggered="${left_tine_camera_rgbd_sim_triggered}"
-                             sim_rgbd_visible_mask="${left_tine_camera_rgbd_sim_visible_mask}"
-                             sim_rgbd_clip="${left_tine_camera_rgbd_sim_clip}"
-                             sim_rgbd_depth_clip="${left_tine_camera_rgbd_sim_depth_clip}"
-                             sim_rgbd_update_rate="${left_tine_camera_rgbd_sim_update_rate}"
-                             sim_rgbd_image="${left_tine_camera_rgbd_sim_image}"
-                             sim_rgbd_lens_single_elements="${left_tine_camera_rgbd_sim_lens_single_elements}"
-                             sim_rgbd_lens_custom_function="${left_tine_camera_rgbd_sim_lens_custom_function}"
-                             sim_rgbd_lens_intrinsics="${left_tine_camera_rgbd_sim_lens_intrinsics}"
-                             sim_rgbd_lens_xy_skew="${left_tine_camera_rgbd_sim_lens_xy_skew}"
-                             sim_rgbd_lens_projection="${left_tine_camera_rgbd_sim_lens_projection}"
-                             sim_rgbd_distortion_k_p="${left_tine_camera_rgbd_sim_distortion_k_p}"
-                             sim_rgbd_distortion_center="${left_tine_camera_rgbd_sim_distortion_center}"
-                             sim_rgbd_gaussian_noise="${left_tine_camera_rgbd_sim_gaussian_noise}"
-                             sim_infra1_enabled="${use_sim_mode and left_tine_camera_infra1_sim_enabled}"
-                             sim_infra1_use_gravity="${left_tine_camera_infra1_sim_use_gravity}"
-                             sim_infra1_always_on="${left_tine_camera_infra1_sim_always_on}"
-                             sim_infra1_visualize="${left_tine_camera_infra1_sim_visualize}"
-                             sim_infra1_enable_metrics="${left_tine_camera_infra1_sim_enable_metrics}"
-                             sim_infra1_save="${left_tine_camera_infra1_sim_save}"
-                             sim_infra1_triggered="${left_tine_camera_infra1_sim_triggered}"
-                             sim_infra1_visible_mask="${left_tine_camera_infra1_sim_visible_mask}"
-                             sim_infra1_clip="${left_tine_camera_infra1_sim_clip}"
-                             sim_infra1_update_rate="${left_tine_camera_infra1_sim_update_rate}"
-                             sim_infra1_image="${left_tine_camera_infra1_sim_image}"
-                             sim_infra1_lens_single_elements="${left_tine_camera_infra1_sim_lens_single_elements}"
-                             sim_infra1_lens_custom_function="${left_tine_camera_infra1_sim_lens_custom_function}"
-                             sim_infra1_lens_intrinsics="${left_tine_camera_infra1_sim_lens_intrinsics}"
-                             sim_infra1_lens_xy_skew="${left_tine_camera_infra1_sim_lens_xy_skew}"
-                             sim_infra1_lens_projection="${left_tine_camera_infra1_sim_lens_projection}"
-                             sim_infra1_distortion_k_p="${left_tine_camera_infra1_sim_distortion_k_p}"
-                             sim_infra1_distortion_center="${left_tine_camera_infra1_sim_distortion_center}"
-                             sim_infra1_gaussian_noise="${left_tine_camera_infra1_sim_gaussian_noise}"
-                             sim_infra2_enabled="${use_sim_mode and left_tine_camera_infra2_sim_enabled}"
-                             sim_infra2_use_gravity="${left_tine_camera_infra2_sim_use_gravity}"
-                             sim_infra2_always_on="${left_tine_camera_infra2_sim_always_on}"
-                             sim_infra2_visualize="${left_tine_camera_infra2_sim_visualize}"
-                             sim_infra2_enable_metrics="${left_tine_camera_infra2_sim_enable_metrics}"
-                             sim_infra2_save="${left_tine_camera_infra2_sim_save}"
-                             sim_infra2_triggered="${left_tine_camera_infra2_sim_triggered}"
-                             sim_infra2_visible_mask="${left_tine_camera_infra2_sim_visible_mask}"
-                             sim_infra2_clip="${left_tine_camera_infra2_sim_clip}"
-                             sim_infra2_update_rate="${left_tine_camera_infra2_sim_update_rate}"
-                             sim_infra2_image="${left_tine_camera_infra2_sim_image}"
-                             sim_infra2_lens_single_elements="${left_tine_camera_infra2_sim_lens_single_elements}"
-                             sim_infra2_lens_custom_function="${left_tine_camera_infra2_sim_lens_custom_function}"
-                             sim_infra2_lens_intrinsics="${left_tine_camera_infra2_sim_lens_intrinsics}"
-                             sim_infra2_lens_xy_skew="${left_tine_camera_infra2_sim_lens_xy_skew}"
-                             sim_infra2_lens_projection="${left_tine_camera_infra2_sim_lens_projection}"
-                             sim_infra2_distortion_k_p="${left_tine_camera_infra2_sim_distortion_k_p}"
-                             sim_infra2_distortion_center="${left_tine_camera_infra2_sim_distortion_center}"
-                             sim_infra2_gaussian_noise="${left_tine_camera_infra2_sim_gaussian_noise}"
-                             sim_rgbd_base_topic="${left_tine_camera_rgbd_sim_base_topic}"
-                             sim_rgbd_trigger_topic="${left_tine_camera_rgbd_sim_trigger_topic}"
-                             sim_infra1_image_topic="${left_tine_camera_infra1_sim_topic}"
-                             sim_infra1_camera_info_topic="${left_tine_camera_infra1_sim_info_topic}"
-                             sim_infra1_trigger_topic="${left_tine_camera_infra1_sim_trigger_topic}"
-                             sim_infra2_image_topic="${left_tine_camera_infra2_sim_topic}"
-                             sim_infra2_camera_info_topic="${left_tine_camera_infra2_sim_info_topic}"
-                             sim_infra2_trigger_topic="${left_tine_camera_infra2_sim_trigger_topic}"/>
-  <!-- ===================================================================== -->
-  <!-- RIGHT TINE CAMERA: REALSENSE D435 -->
-  <!-- ===================================================================== -->
-  <xacro:property name="right_tine_rgbd_use_visual"       value="$(arg right_tine_rgbd_use_visual)"/>
-  <xacro:property name="right_tine_rgbd_use_collision"    value="$(arg right_tine_rgbd_use_collision)"/>
-  <xacro:property name="right_tine_rgbd_use_inertial"     value="$(arg right_tine_rgbd_use_inertial)"/>
-  <xacro:property name="right_tine_rgbd_use_v_mesh"       value="$(arg right_tine_rgbd_use_v_mesh)"/>
-  <xacro:property name="right_tine_rgbd_color"            value="$(arg right_tine_rgbd_color)"/>
-  <xacro:property name="right_tine_rgbd_use_c_mesh"       value="$(arg right_tine_rgbd_use_c_mesh)"/>
-  <xacro:property name="right_tine_camera_rgbd_sim_cfg"   value="${sim_cfg.get('right_tine_camera_rgbd', dict())}"/>
-  <xacro:property name="right_tine_camera_infra1_sim_cfg" value="${sim_cfg.get('right_tine_camera_infra1', dict())}"/>
-  <xacro:property name="right_tine_camera_infra2_sim_cfg" value="${sim_cfg.get('right_tine_camera_infra2', dict())}"/>
-  <!-- Set properties for the `rgbd_camera` Gazebo plugin associated to the right tine camera. -->
-  <xacro:set_props_plugin_camera_rgbd prop_prefix="right_tine_camera_rgbd_sim"
-                                      sim_cfg="${right_tine_camera_rgbd_sim_cfg}"/>
-  <!-- Set properties for the first infrared Gazebo plugin in the right tine camera. -->
-  <xacro:set_props_plugin_camera prop_prefix="right_tine_camera_infra1_sim"
-                                 sim_cfg="${right_tine_camera_infra1_sim_cfg}"/>
-  <!-- Set properties for the second infrared Gazebo plugin in the right tine camera. -->
-  <xacro:set_props_plugin_camera prop_prefix="right_tine_camera_infra2_sim"
-                                 sim_cfg="${right_tine_camera_infra2_sim_cfg}"/>
-  <!--
-  The right tine camera uses the same x and z coordinates as the left tine camera.
-  The y coordinate is mirrored around the tine center line.
-  -->
-  <xacro:property name="right_tine_rgbd_mount_x" value="${left_tine_rgbd_mount_x}"/>
-  <xacro:property name="right_tine_rgbd_mount_y" value="${-left_tine_rgbd_mount_y}"/>
-  <xacro:property name="right_tine_rgbd_mount_z" value="${left_tine_rgbd_mount_z}"/>
-  <xacro:realsense_d435_rgbd name="right_tine_camera"
-                             prefix="${robot_prefix}"
-                             namespace="${robot_namespace}"
-                             parent_frame="${robot_prefix}${fork_name}_right_tine_link"
-                             use_visual="${right_tine_rgbd_use_visual}"
-                             use_collision="${right_tine_rgbd_use_collision}"
-                             use_inertial="${right_tine_rgbd_use_inertial}"
-                             use_v_mesh="${right_tine_rgbd_use_v_mesh}"
-                             color="${right_tine_rgbd_color}"
-                             use_c_mesh="${right_tine_rgbd_use_c_mesh}"
-                             joint_parent_fr_root_fr="${right_tine_rgbd_mount_x} ${right_tine_rgbd_mount_y} ${right_tine_rgbd_mount_z} 0.0 0.0 0.0"
-                             use_sensor_frames_and_joints="${use_sim_mode}"
-                             sim_rgbd_enabled="${use_sim_mode and right_tine_camera_rgbd_sim_enabled}"
-                             sim_rgbd_use_gravity="${right_tine_camera_rgbd_sim_use_gravity}"
-                             sim_rgbd_always_on="${right_tine_camera_rgbd_sim_always_on}"
-                             sim_rgbd_visualize="${right_tine_camera_rgbd_sim_visualize}"
-                             sim_rgbd_enable_metrics="${right_tine_camera_rgbd_sim_enable_metrics}"
-                             sim_rgbd_save="${right_tine_camera_rgbd_sim_save}"
-                             sim_rgbd_triggered="${right_tine_camera_rgbd_sim_triggered}"
-                             sim_rgbd_visible_mask="${right_tine_camera_rgbd_sim_visible_mask}"
-                             sim_rgbd_clip="${right_tine_camera_rgbd_sim_clip}"
-                             sim_rgbd_depth_clip="${right_tine_camera_rgbd_sim_depth_clip}"
-                             sim_rgbd_update_rate="${right_tine_camera_rgbd_sim_update_rate}"
-                             sim_rgbd_image="${right_tine_camera_rgbd_sim_image}"
-                             sim_rgbd_lens_single_elements="${right_tine_camera_rgbd_sim_lens_single_elements}"
-                             sim_rgbd_lens_custom_function="${right_tine_camera_rgbd_sim_lens_custom_function}"
-                             sim_rgbd_lens_intrinsics="${right_tine_camera_rgbd_sim_lens_intrinsics}"
-                             sim_rgbd_lens_xy_skew="${right_tine_camera_rgbd_sim_lens_xy_skew}"
-                             sim_rgbd_lens_projection="${right_tine_camera_rgbd_sim_lens_projection}"
-                             sim_rgbd_distortion_k_p="${right_tine_camera_rgbd_sim_distortion_k_p}"
-                             sim_rgbd_distortion_center="${right_tine_camera_rgbd_sim_distortion_center}"
-                             sim_rgbd_gaussian_noise="${right_tine_camera_rgbd_sim_gaussian_noise}"
-                             sim_infra1_enabled="${use_sim_mode and right_tine_camera_infra1_sim_enabled}"
-                             sim_infra1_use_gravity="${right_tine_camera_infra1_sim_use_gravity}"
-                             sim_infra1_always_on="${right_tine_camera_infra1_sim_always_on}"
-                             sim_infra1_visualize="${right_tine_camera_infra1_sim_visualize}"
-                             sim_infra1_enable_metrics="${right_tine_camera_infra1_sim_enable_metrics}"
-                             sim_infra1_save="${right_tine_camera_infra1_sim_save}"
-                             sim_infra1_triggered="${right_tine_camera_infra1_sim_triggered}"
-                             sim_infra1_visible_mask="${right_tine_camera_infra1_sim_visible_mask}"
-                             sim_infra1_clip="${right_tine_camera_infra1_sim_clip}"
-                             sim_infra1_update_rate="${right_tine_camera_infra1_sim_update_rate}"
-                             sim_infra1_image="${right_tine_camera_infra1_sim_image}"
-                             sim_infra1_lens_single_elements="${right_tine_camera_infra1_sim_lens_single_elements}"
-                             sim_infra1_lens_custom_function="${right_tine_camera_infra1_sim_lens_custom_function}"
-                             sim_infra1_lens_intrinsics="${right_tine_camera_infra1_sim_lens_intrinsics}"
-                             sim_infra1_lens_xy_skew="${right_tine_camera_infra1_sim_lens_xy_skew}"
-                             sim_infra1_lens_projection="${right_tine_camera_infra1_sim_lens_projection}"
-                             sim_infra1_distortion_k_p="${right_tine_camera_infra1_sim_distortion_k_p}"
-                             sim_infra1_distortion_center="${right_tine_camera_infra1_sim_distortion_center}"
-                             sim_infra1_gaussian_noise="${right_tine_camera_infra1_sim_gaussian_noise}"
-                             sim_infra2_enabled="${use_sim_mode and right_tine_camera_infra2_sim_enabled}"
-                             sim_infra2_use_gravity="${right_tine_camera_infra2_sim_use_gravity}"
-                             sim_infra2_always_on="${right_tine_camera_infra2_sim_always_on}"
-                             sim_infra2_visualize="${right_tine_camera_infra2_sim_visualize}"
-                             sim_infra2_enable_metrics="${right_tine_camera_infra2_sim_enable_metrics}"
-                             sim_infra2_save="${right_tine_camera_infra2_sim_save}"
-                             sim_infra2_triggered="${right_tine_camera_infra2_sim_triggered}"
-                             sim_infra2_visible_mask="${right_tine_camera_infra2_sim_visible_mask}"
-                             sim_infra2_clip="${right_tine_camera_infra2_sim_clip}"
-                             sim_infra2_update_rate="${right_tine_camera_infra2_sim_update_rate}"
-                             sim_infra2_image="${right_tine_camera_infra2_sim_image}"
-                             sim_infra2_lens_single_elements="${right_tine_camera_infra2_sim_lens_single_elements}"
-                             sim_infra2_lens_custom_function="${right_tine_camera_infra2_sim_lens_custom_function}"
-                             sim_infra2_lens_intrinsics="${right_tine_camera_infra2_sim_lens_intrinsics}"
-                             sim_infra2_lens_xy_skew="${right_tine_camera_infra2_sim_lens_xy_skew}"
-                             sim_infra2_lens_projection="${right_tine_camera_infra2_sim_lens_projection}"
-                             sim_infra2_distortion_k_p="${right_tine_camera_infra2_sim_distortion_k_p}"
-                             sim_infra2_distortion_center="${right_tine_camera_infra2_sim_distortion_center}"
-                             sim_infra2_gaussian_noise="${right_tine_camera_infra2_sim_gaussian_noise}"
-                             sim_rgbd_base_topic="${right_tine_camera_rgbd_sim_base_topic}"
-                             sim_rgbd_trigger_topic="${right_tine_camera_rgbd_sim_trigger_topic}"
-                             sim_infra1_image_topic="${right_tine_camera_infra1_sim_topic}"
-                             sim_infra1_camera_info_topic="${right_tine_camera_infra1_sim_info_topic}"
-                             sim_infra1_trigger_topic="${right_tine_camera_infra1_sim_trigger_topic}"
-                             sim_infra2_image_topic="${right_tine_camera_infra2_sim_topic}"
-                             sim_infra2_camera_info_topic="${right_tine_camera_infra2_sim_info_topic}"
-                             sim_infra2_trigger_topic="${right_tine_camera_infra2_sim_trigger_topic}"/>
   <xacro:if value="${use_sim_mode}">
     <gazebo>
